Commit message: simple model in rviz and gazebo

File: urdf/human/chest_included_npose_inertia.xacro (robot description, xacro)
@@ -10,5 +10,44 @@
     <color rgba="1 1 1 1"/>
   </material>
+  <xacro:property name="l_neck" value="0.053" />
+  <xacro:property name="head" value="0.212-${neck}" />
+  <xacro:property name="l_upper_trunk" value="0.410" />
+  <xacro:property name="l_lower_trunk" value="0.135" />
+  <xacro:property name="l_upper_arm" value="0.65" />
+  <xacro:property name="l_forearm" value="0.299" />
+  <xacro:property name="l_hand" value="0.203" />
+  <xacro:property name="l_thigh" value="0.449" />
+  <xacro:property name="l_shank" value="0.429" />
+  <xacro:property name="l_foot" value="0.06" />
+  <xacro:property name="whole_body" value="1.7268" />
+  <xacro:property name="w_neck" value="${l_neck/5}" />
+  <xacro:property name="w_upper_trunk" value="${l_upper_trunk/5}" />
+  <xacro:property name="w_lower_trunk" value="${l_lower_trunk/2}" />
+  <xacro:property name="w_upper_arm" value="${l_upper_arm/3}" />
+  <xacro:property name="w_forearm" value="${l_forearm/3}" />
+  <xacro:property name="w_hand" value="${l_hand/3}" />
+  <xacro:property name="w_thigh" value="${l_thigh/3}" />
+  <xacro:property name="w_shank" value="${l_shank/3}" />
+  <xacro:property name="w_foot" value="${l_foot/3}" />
+  <xacro:property name="cm_head" value="0.361" />
+  <xacro:property name="cm_upper_trunk" value="0.497" />
+  <xacro:property name="cm_lower_trunk" value="0.518" />
+  <xacro:property name="cm_upper_arm" value="0.427" />
+  <xacro:property name="cm_forearm" value="0.417" />
+  <xacro:property name="cm_hand" value="0.361" />
+  <xacro:property name="cm_thigh" value="0.430" />
+  <xacro:property name="cm_shank" value="0.443" />
+  <xacro:property name="cm_foot" value="0.436" />
+  <xacro:property name="d_head" value="1085.1" />
+  <xacro:property name="d_upper_trunk" value="1068.6" />
+  <xacro:property name="d_lower_trunk" value="1068.6" />
+  <xacro:property name="d_upper_arm" value="1088.0" />
+  <xacro:property name="d_forearm" value="1108.6" />
+  <xacro:property name="d_hand" value="1112.6" />
+  <xacro:property name="d_thigh" value="1068.6" />
+  <xacro:property name="d_shank" value="1100.2" />
+  <xacro:property name="d_foot" value="1089.3" />
   <xacro:include filename="spherical.urdf.xacro"/>
+  <xacro:include filename="arm.urdf.xacro"/>
   <create/>
   <link name="world"/>
@@ -16,5 +55,5 @@
     <parent link="world"/>
     <child link="base_link"/>
-    <origin rpy="0.0 0.0 0.0" xyz="0 0 1.05"/>
+    <origin rpy="0.0 0.0 0.0" xyz="0 0 ${l_foot+l_shank+l_thigh+l_lower_trunk}"/>
   </joint>
   <link name="base_link">
@@ -27,461 +66,39 @@
     </visual>
   </link>
+  <!--<xacro:spherical name="joint_1" parent="base_link" child="link_01">
+    <origin rpy="0 0 0" xyz="0 0 0"/>
+  </xacro:spherical>-->
   <joint name="human_base" type="fixed">
     <origin rpy="0 0 0" xyz="0 0 0"/>
     <parent link="base_link"/>
-    <child link="human/base"/>
+    <child link="link_02"/>
   </joint>
-  <link name="human/base">
-    <visual>
-      <origin rpy="0 0 0" xyz="0 0 -0.0405569060538"/>
-      <geometry>
-        <cylinder length="-0.0811138121076" radius="0.130553532998"/>
-      </geometry>
-    </visual>
-  </link>
-  <link name="human/spine_0">
-    <visual>
-      <origin rpy="0 0 0" xyz="0 0 0.0363124478192"/>
-      <geometry>
-        <cylinder length="0.0726248956383" radius="0.141172520845"/>
-      </geometry>
-    </visual>
-  </link>
-  <link name="human/spine_1"/>
-  <link name="human/spine_2"/>
-  <link name="human/spine">
-    <visual>
-      <origin rpy="0 0 0" xyz="0 0 0.137944030927"/>
-      <geometry>
-        <cylinder length="0.275888061853" radius="0.161172520845"/>
-      </geometry>
-    </visual>
-  </link>
-  <link name="human/shoulder_center">
-    <visual>
-      <origin rpy="0 0 0" xyz="0 0 0.050635057485"/>
-      <geometry>
-        <cylinder length="0.10127011497" radius="0.181172520845"/>
-      </geometry>
-    </visual>
-  </link>
-  <link name="human/neck_0"/>
-  <link name="human/neck_1"/>
-  <link name="human/neck">
-    <visual>
-      <origin rpy="0 0 0" xyz="0 0 0.102139711472"/>
-      <geometry>
-        <cylinder length="0.204279422944" radius="0.04"/>
-      </geometry>
-    </visual>
-  </link>
-  <link name="human/head">
-    <visual>
-      <origin rpy="0 0 0" xyz="0 0 0"/>
-      <geometry>
-        <sphere radius="0.1"/>
-      </geometry>
-    </visual>
-  </link>
-  <joint name="hip" type="fixed">
+  <!--<xacro:cylindrical_part name="link_02" density="1" cm="1" length="5" radius="2">
     <origin rpy="0 0 0" xyz="0 0 0"/>
-    <parent link="human/base"/>
-    <child link="human/spine_0"/>
-  </joint>
-  <!-- SPINE : spherical -->
-  <joint name="spine_0" type="revolute">
-    <origin rpy="0 0 0" xyz="0 0 0.0726248956383"/>
-    <axis xyz="1 0 0"/>
-    <parent link="human/spine_0"/>
-    <child link="human/spine_1"/>
-    <limit effort="1" lower="-1.57079632679" upper="1.57079632679" velocity="1"/>
-  </joint>
-  <joint name="spine_1" type="revolute">
-    <origin rpy="0 0 0" xyz="0 0 0"/>
-    <axis xyz="0 1 0"/>
-    <parent link="human/spine_1"/>
-    <child link="human/spine_2"/>
-    <limit effort="1" lower="-1.57079632679" upper="1.57079632679" velocity="1"/>
-  </joint>
-  <joint name="spine_2" type="revolute">
-    <origin rpy="0 0 0" xyz="0 0 0"/>
-    <axis xyz="0 0 1"/>
-    <parent link="human/spine_2"/>
-    <child link="human/spine"/>
-    <limit effort="1" lower="-1.57079632679" upper="1.57079632679" velocity="1"/>
-  </joint>
-  <joint name="shoulder_center" type="fixed">
-    <origin rpy="0 0 0" xyz="0 0 0.275888061853"/>
-    <parent link="human/spine"/>
-    <child link="human/shoulder_center"/>
-  </joint>
-  <!-- NECK : spherical -->
-  <joint name="neck_0" type="fixed">
-    <origin rpy="0 0 0" xyz="0 0 0.10127011497"/>
-    <parent link="human/shoulder_center"/>
-    <child link="human/neck_0"/>
-  </joint>
-  <joint name="neck_1" type="fixed">
-    <origin rpy="0 0 0" xyz="0 0 0"/>
-    <parent link="human/neck_0"/>
-    <child link="human/neck_1"/>
-  </joint>
-  <joint name="neck_2" type="fixed">
-    <origin rpy="0 0 0" xyz="0 0 0"/>
-    <parent link="human/neck_1"/>
-    <child link="human/neck"/>
-  </joint>
-  <!-- END NECK -->
-  <joint name="head" type="fixed">
-    <origin rpy="0 0 0" xyz="0 0 0.204279422944"/>
-    <parent link="human/neck"/>
-    <child link="human/head"/>
-  </joint>
-  <link name="human/right_arm_mount"/>
-  <link name="human/right_shoulder_0"/>
-  <link name="human/right_shoulder_1"/>
-  <link name="human/right_shoulder">
-    <visual>
-      <origin rpy="0 1.57079632679 0" xyz="0.147075804738 0 0"/>
-      <geometry>
-        <cylinder length="0.294151609476" radius="0.05"/>
-      </geometry>
-    </visual>
-  </link>
-  <link name="human/right_elbow_0"/>
-  <link name="human/right_elbow">
-    <visual>
-      <origin rpy="0 1.57079632679 0" xyz="0.137074736994 0 0"/>
-      <geometry>
-        <cylinder length="0.274149473988" radius="0.025"/>
-      </geometry>
-    </visual>
-  </link>
-  <link name="human/right_wrist_0"/>
-  <link name="human/right_wrist_1"/>
-  <link name="human/right_wrist">
-    <visual>
-      <origin rpy="0 0 0" xyz="0.05 0 0"/>
-      <geometry>
-        <box size="0.1 0.05 .005"/>
-      </geometry>
-    </visual>
-  </link>
-  <link name="human/right_hand"/>
-  <!-- Joints -->
-  <joint name="right_arm_mount" type="fixed">
-    <origin rpy="0 1.57079632679 -1.57079632679" xyz="0 -0.181172520845 -0.00609526854636"/>
-    <parent link="human/shoulder_center"/>
-    <child link="human/right_arm_mount"/>
-  </joint>
-  <!-- SHOULDER : spherical -->
-  <joint name="right_shoulder_0" type="revolute">
-    <origin rpy="0 0 0" xyz="0 0 0"/>
-    <axis xyz="0 0 1"/>
-    <parent link="human/right_arm_mount"/>
-    <child link="human/right_shoulder_0"/>
-    <limit effort="1" lower="-1.57079632679" upper="1.57079632679" velocity="1"/>
-  </joint>
-  <joint name="right_shoulder_1" type="revolute">
-    <origin rpy="0 0 0" xyz="0 0 0"/>
-    <axis xyz="0 -1 0"/>
-    <parent link="human/right_shoulder_0"/>
-    <child link="human/right_shoulder_1"/>
-    <limit effort="1" lower="-1.57079632679" upper="2.35619449019" velocity="1"/>
-  </joint>
-  <joint name="right_shoulder_2" type="revolute">
-    <origin rpy="0 0 0" xyz="0 0 0"/>
-    <axis xyz="1 0 0"/>
-    <parent link="human/right_shoulder_1"/>
-    <child link="human/right_shoulder"/>
-    <limit effort="1" lower="-1.57079632679" upper="1.57079632679" velocity="1"/>
-  </joint>
-  <!-- END SHOULDER -->
-  <joint name="right_elbow_0" type="revolute">
-    <origin rpy="0 0 0" xyz="0.294151609476 0 0"/>
-    <axis xyz="0 0 1"/>
-    <parent link="human/right_shoulder"/>
-    <child link="human/right_elbow_0"/>
-    <limit effort="1" lower="-3.14159265359" upper="3.14159265359" velocity="1"/>
-  </joint>
-  <joint name="right_elbow_2" type="revolute">
-    <origin rpy="0 0 0" xyz="0 0 0"/>
-    <axis xyz="1 0 0"/>
-    <parent link="human/right_elbow_0"/>
-    <child link="human/right_elbow"/>
-    <limit effort="1" lower="0.0" upper="1.57079632679" velocity="1"/>
-  </joint>
-  <joint name="right_wrist_0" type="fixed">
-    <origin rpy="0 0 0" xyz="0.274149473988 0 0"/>
-    <axis xyz="0 1 0"/>
-    <parent link="human/right_elbow"/>
-    <child link="human/right_wrist_0"/>
-    <limit effort="1" lower="-0.78539816339" upper="0.78539816339" velocity="1"/>
-  </joint>
-  <joint name="right_wrist_1" type="fixed">
-    <origin rpy="0 0 0" xyz="0 0 0"/>
-    <axis xyz="0 0 1"/>
-    <parent link="human/right_wrist_0"/>
-    <child link="human/right_wrist_1"/>
-    <limit effort="1" lower="-1.57079632679" upper="1.57079632679" velocity="1"/>
-  </joint>
-  <joint name="right_wrist_2" type="fixed">
-    <origin rpy="0 0 0" xyz="0 0 0"/>
-    <axis xyz="1 0 0"/>
-    <parent link="human/right_wrist_1"/>
-    <child link="human/right_wrist"/>
-    <limit effort="1" lower="-1.57079632679" upper="1.57079632679" velocity="1"/>
-  </joint>
-  <joint name="right_hand" type="fixed">
-    <origin rpy="0 0 0" xyz="0.1 0 0"/>
-    <parent link="human/right_wrist"/>
-    <child link="human/right_hand"/>
-  </joint>
-  <link name="human/left_arm_mount"/>
-  <link name="human/left_shoulder_0"/>
-  <link name="human/left_shoulder_1"/>
-  <link name="human/left_shoulder">
-    <visual>
-      <origin rpy="0 1.57079632679 0" xyz="0.147075804738 0 0"/>
-      <geometry>
-        <cylinder length="0.294151609476" radius="0.05"/>
-      </geometry>
-    </visual>
-  </link>
-  <link name="human/left_elbow_0"/>
-  <link name="human/left_elbow">
-    <visual>
-      <origin rpy="0 1.57079632679 0" xyz="0.137074736994 0 0"/>
-      <geometry>
-        <cylinder length="0.274149473988" radius="0.025"/>
-      </geometry>
-    </visual>
-  </link>
-  <link name="human/left_wrist_0"/>
-  <link name="human/left_wrist_1"/>
-  <link name="human/left_wrist">
-    <visual>
-      <origin rpy="0 0 0" xyz="0.05 0 0"/>
-      <geometry>
-        <box size="0.1 0.05 .005"/>
-      </geometry>
-    </visual>
-  </link>
-  <link name="human/left_hand"/>
-  <!-- Joints -->
-  <joint name="left_arm_mount" type="fixed">
-    <origin rpy="0 1.57079632679 1.57079632679" xyz="0 0.181172520845 -0.00609526854636"/>
-    <parent link="human/shoulder_center"/>
-    <child link="human/left_arm_mount"/>
-  </joint>
-  <!-- SHOULDER : spherical -->
-  <joint name="left_shoulder_0" type="revolute">
-    <origin rpy="0 0 0" xyz="0 0 0"/>
-    <axis xyz="0 0 -1"/>
-    <parent link="human/left_arm_mount"/>
-    <child link="human/left_shoulder_0"/>
-    <limit effort="1" lower="-1.57079632679" upper="1.57079632679" velocity="1"/>
-  </joint>
-  <joint name="left_shoulder_1" type="revolute">
-    <origin rpy="0 0 0" xyz="0 0 0"/>
-    <axis xyz="0 -1 0"/>
-    <parent link="human/left_shoulder_0"/>
-    <child link="human/left_shoulder_1"/>
-    <limit effort="1" lower="-1.57079632679" upper="2.35619449019" velocity="1"/>
-  </joint>
-  <joint name="left_shoulder_2" type="revolute">
-    <origin rpy="0 0 0" xyz="0 0 0"/>
-    <parent link="human/left_shoulder_1"/>
-    <child link="human/left_shoulder"/>
-    <limit effort="1" lower="-1.57079632679" upper="1.57079632679" velocity="1"/>
-  </joint>
-  <!-- END SHOULDER -->
-  <joint name="left_elbow_0" type="revolute">
-    <origin rpy="0 0 0" xyz="0.294151609476 0 0"/>
-    <axis xyz="0 0 -1"/>
-    <parent link="human/left_shoulder"/>
-    <child link="human/left_elbow_0"/>
-    <limit effort="1" lower="-3.14159265359" upper="3.14159265359" velocity="1"/>
-  </joint>
-  <joint name="left_elbow_2" type="revolute">
-    <origin rpy="0 0 0" xyz="0 0 0"/>
-    <axis xyz="-1 0 0"/>
-    <parent link="human/left_elbow_0"/>
-    <child link="human/left_elbow"/>
-    <limit effort="1" lower="0.0" upper="1.57079632679" velocity="1"/>
-  </joint>
-  <joint name="left_wrist_0" type="revolute">
-    <origin rpy="0 0 0" xyz="0.274149473988 0 0"/>
-    <axis xyz="0 1 0"/>
-    <parent link="human/left_elbow"/>
-    <child link="human/left_wrist_0"/>
-    <limit effort="1" lower="-0.78539816339" upper="0.78539816339" velocity="1"/>
-  </joint>
-  <joint name="left_wrist_1" type="revolute">
-    <origin rpy="0 0 0" xyz="0 0 0"/>
-    <axis xyz="0 0 1"/>
-    <parent link="human/left_wrist_0"/>
-    <child link="human/left_wrist_1"/>
-    <limit effort="1" lower="-1.57079632679" upper="1.57079632679" velocity="1"/>
-  </joint>
-  <joint name="left_wrist_2" type="revolute">
-    <origin rpy="0 0 0" xyz="0 0 0"/>
-    <axis xyz="1 0 0"/>
-    <parent link="human/left_wrist_1"/>
-    <child link="human/left_wrist"/>
-    <limit effort="1" lower="-1.57079632679" upper="1.57079632679" velocity="1"/>
-  </joint>
-  <joint name="left_hand" type="fixed">
-    <origin rpy="0 0 0" xyz="0.1 0 0"/>
-    <parent link="human/left_wrist"/>
-    <child link="human/left_hand"/>
-  </joint>
-  <link name="human/right_leg_mount"/>
-  <link name="human/right_hip_0"/>
-  <link name="human/right_hip_1"/>
-  <link name="human/right_hip">
-    <visual>
-      <origin rpy="0 1.57079632679 0" xyz="0.282210946758 0 0"/>
-      <geometry>
-        <cylinder length="0.564421893516" radius="0.05"/>
-      </geometry>
-    </visual>
-  </link>
-  <link name="human/right_knee">
-    <visual>
-      <origin rpy="0 1.57079632679 0" xyz="0.203668548616 0 0"/>
-      <geometry>
-        <cylinder length="0.407337097232" radius="0.025"/>
-      </geometry>
-    </visual>
-  </link>
-  <link name="human/right_ankle_0"/>
-  <link name="human/right_ankle">
-    <visual>
-      <origin rpy="0 0 0" xyz="0.05 0 0"/>
-      <geometry>
-        <box size="0.1 0.05 .005"/>
-      </geometry>
-    </visual>
-  </link>
-  <link name="human/right_foot"/>
-  <!-- Joints -->
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
Commit message: noetic update for joint state publisher

File: urdf/human/chest_included_npose_inertia.xacro (robot description, xacro)
@@ -1,4 +1,7 @@
 <?xml version="1.0" ?>
 <robot name="human_upper" xmlns:xacro="http://www.ros.org/wiki/xacro">
+  <gazebo>
+    <static>false</static>
+  </gazebo>
   <material name="blue">
     <color rgba="0 0 0.8 1"/>
@@ -55,5 +58,5 @@
     <parent link="world"/>
     <child link="base_link"/>
-    <origin rpy="0.0 0.0 0.0" xyz="0 0 ${l_foot+l_shank+l_thigh+l_lower_trunk}"/>
+    <origin rpy="0.0 0.0 0.0" xyz="0 0 0"/>
   </joint>
   <link name="base_link">
@@ -61,44 +64,27 @@
       <origin rpy="0 0 0" xyz="0 0 0"/>
       <geometry>
-        <sphere radius="0.1"/>
+        <box size="1 1 1"/>
       </geometry>
-      <material name="white"/>
     </visual>
   </link>
-  <!--<xacro:spherical name="joint_1" parent="base_link" child="link_01">
-    <origin rpy="0 0 0" xyz="0 0 0"/>
-  </xacro:spherical>-->
-  <joint name="human_base" type="fixed">
-    <origin rpy="0 0 0" xyz="0 0 0"/>
+  <joint name="base_link__link_01" type="revolute">
+    <axis xyz="1 0 0" rpy="0 0 0"/>
+    <limit effort="1000.0" lower="-3.14" upper="3.14" velocity="0.5"/>
+    <origin rpy="0 0 0" xyz="0 0 0.5"/>
     <parent link="base_link"/>
-    <child link="link_02"/>
+    <child link="link_01"/>
   </joint>
-  <!--<xacro:cylindrical_part name="link_02" density="1" cm="1" length="5" radius="2">
-    <origin rpy="0 0 0" xyz="0 0 0"/>
-  </xacro:cylindrical_part>-->
-  <xacro:property name="mass" value="${pi*l_upper_arm*pow(w_upper_arm,2)*d_upper_arm}" />
-  <link name="link_02">
-      <visual>
-        <origin xyz="0 0 0" rpy="0 0 0" />
-        <geometry>
-          <!--<mesh filename="package://pr2_description/meshes/torso_v0/torso_lift.dae"  /> -->
-          <cylinder length="${l_upper_arm}" radius="${w_upper_arm}"/>
-        </geometry>
-        <material name="blue" />
-      </visual>
-      <collision>
-        <origin xyz="0 0 0" rpy="0 0 0"/>
-        <geometry>
-          <cylinder length="${l_upper_arm}" radius="${w_upper_arm}"/>
-        </geometry>
-      </collision>
-      <inertial>
-        <origin xyz="0 0 0" rpy="0 0 0"/>
-        <mass value="${mass}"/>
-        <inertia
-          ixx="${mass*(3*pow(w_upper_arm,2)+pow(l_upper_arm,2))/12}" ixy="0.0" ixz="0.0"
-          iyy="${mass*(3*pow(w_upper_arm,2)+pow(l_upper_arm,2))/12}" iyz="0.0"
-          izz="${mass*pow(w_upper_arm,2)/2}"/>
-      </inertial>
-    </link>
+  <!-- <joint name="base_link__link_01" type="fixed">
+    <parent link="base_link"/>
+    <child link="link_01"/>
+    <origin rpy="0.0 0.0 0.0" xyz="0 0 0"/>
+  </joint> -->
+  <link name="link_01">
+    <visual>
+      <origin rpy="0 0 0" xyz="0 0 0.5"/>
+      <geometry>
+        <cylinder radius="0.35" length="0.4"/>
+      </geometry>
+    </visual>
+  </link>
 </robot>

Commit message: temp gazebo and rviz to set controllers

File: urdf/human/chest_included_npose_inertia.xacro (robot description, xacro)
@@ -2,5 +2,5 @@
 <robot name="human_upper" xmlns:xacro="http://www.ros.org/wiki/xacro">
   <gazebo>
-    <static>false</static>
+    <static>true</static>
   </gazebo>
   <material name="blue">
@@ -54,9 +54,11 @@
   <xacro:include filename="arm.urdf.xacro"/>
   <create/>
+  <xacro:property name="mass" value="${pi*l_upper_arm*pow(w_upper_arm,2)*d_upper_arm}" />
   <link name="world"/>
   <joint name="world_joint" type="fixed">
     <parent link="world"/>
     <child link="base_link"/>
-    <origin rpy="0.0 0.0 0.0" xyz="0 0 0"/>
+    <!-- <origin rpy="0.0 0.0 0.0" xyz="0 0 ${l_foot+l_shank+l_thigh+l_lower_trunk}"/> -->
+    <origin rpy="0.0 0.0 0.0" xyz="0 0 0.05"/>
   </joint>
   <link name="base_link">
@@ -64,27 +66,52 @@
       <origin rpy="0 0 0" xyz="0 0 0"/>
       <geometry>
-        <box size="1 1 1"/>
+        <sphere radius="0.1"/>
       </geometry>
+      <material name="white"/>
     </visual>
+    <collision>
+      <origin xyz="0 0 0" rpy="0 0 0"/>
+      <geometry>
+        <sphere radius="0.1"/>
+      </geometry>
+    </collision>
+    <inertial>
+      <origin xyz="0 0 0" rpy="0 0 0"/>
+      <mass value="${mass}"/>
+      <inertia
+        ixx="${mass*(3*pow(w_upper_arm,2)+pow(l_upper_arm,2))/12}" ixy="0.0" ixz="0.0"
+        iyy="${mass*(3*pow(w_upper_arm,2)+pow(l_upper_arm,2))/12}" iyz="0.0"
+        izz="${mass*pow(w_upper_arm,2)/2}"/>
+    </inertial>
   </link>
-  <joint name="base_link__link_01" type="revolute">
-    <axis xyz="1 0 0" rpy="0 0 0"/>
-    <limit effort="1000.0" lower="-3.14" upper="3.14" velocity="0.5"/>
-    <origin rpy="0 0 0" xyz="0 0 0.5"/>
-    <parent link="base_link"/>
-    <child link="link_01"/>
-  </joint>
-  <!-- <joint name="base_link__link_01" type="fixed">
-    <parent link="base_link"/>
-    <child link="link_01"/>
-    <origin rpy="0.0 0.0 0.0" xyz="0 0 0"/>
-  </joint> -->
+  <xacro:spherical name="joint_1" parent="base_link" child="link_01">
+    <origin rpy="0 0 0" xyz="0 0 0"/>
+  </xacro:spherical>
+  <!--<xacro:cylindrical_part name="link_02" density="1" cm="1" length="5" radius="2">
+    <origin rpy="0 0 0" xyz="0 0 0"/>
+  </xacro:cylindrical_part>-->
   <link name="link_01">
-    <visual>
-      <origin rpy="0 0 0" xyz="0 0 0.5"/>
-      <geometry>
-        <cylinder radius="0.35" length="0.4"/>
-      </geometry>
-    </visual>
-  </link>
+      <visual>
+        <origin xyz="0 0 0" rpy="0 0 0" />
+        <geometry>
+          <!--<mesh filename="package://pr2_description/meshes/torso_v0/torso_lift.dae"  /> -->
+          <cylinder length="${l_upper_arm}" radius="${w_upper_arm}"/>
+        </geometry>
+        <material name="blue" />
+      </visual>
+      <collision>
+        <origin xyz="0 0 0" rpy="0 0 0"/>
+        <geometry>
+          <cylinder length="${l_upper_arm}" radius="${w_upper_arm}"/>
+        </geometry>
+      </collision>
+      <inertial>
+        <origin xyz="0 0 0" rpy="0 0 0"/>
+        <mass value="${mass}"/>
+        <inertia
+          ixx="${mass*(3*pow(w_upper_arm,2)+pow(l_upper_arm,2))/12}" ixy="0.0" ixz="0.0"
+          iyy="${mass*(3*pow(w_upper_arm,2)+pow(l_upper_arm,2))/12}" iyz="0.0"
+          izz="${mass*pow(w_upper_arm,2)/2}"/>
+      </inertial>
+    </link>
 </robot>

Commit message: xacro update. clean up a bit

File: urdf/human/chest_included_npose_inertia.xacro (robot description, xacro)
@@ -93,5 +93,5 @@
   <link name="link_01">
       <visual>
-        <origin xyz="0 0 0" rpy="0 0 0" />
+        <origin xyz="0 0 ${l_upper_arm/2}" rpy="0 0 0" />
         <geometry>
           <!--<mesh filename="package://pr2_description/meshes/torso_v0/torso_lift.dae"  /> -->
