Commit message: a bit more clean up and controller added (not working tho)

File: urdf/human/human.urdf.xacro (robot description, xacro)
@@ -1,54 +1,11 @@
 <?xml version="1.0" ?>
 <robot name="human" xmlns:xacro="http://www.ros.org/wiki/xacro">
+  <xacro:include filename="$(find imu_human_pkg)/urdf/macros/measurements.xacro" />
+  <xacro:include filename="$(find imu_human_pkg)/urdf/macros/materials.xacro" />
+  <xacro:include filename="$(find imu_human_pkg)/urdf/macros/human.gazebo.xacro" />
+  <xacro:include filename="$(find imu_human_pkg)/urdf/macros/human.transmission.xacro" />
   <gazebo>
     <static>true</static>
   </gazebo>
-  <material name="blue">
-    <color rgba="0 0 0.8 1"/>
-  </material>
-  <material name="black">
-    <color rgba="0 0 0 1"/>
-  </material>
-  <material name="white">
-    <color rgba="1 1 1 1"/>
-  </material>
-  <xacro:property name="l_neck" value="0.053" />
-  <xacro:property name="head" value="0.212-${neck}" />
-  <xacro:property name="l_upper_trunk" value="0.410" />
-  <xacro:property name="l_lower_trunk" value="0.135" />
-  <xacro:property name="l_upper_arm" value="0.65" />
-  <xacro:property name="l_forearm" value="0.299" />
-  <xacro:property name="l_hand" value="0.203" />
-  <xacro:property name="l_thigh" value="0.449" />
-  <xacro:property name="l_shank" value="0.429" />
-  <xacro:property name="l_foot" value="0.06" />
-  <xacro:property name="whole_body" value="1.7268" />
-  <xacro:property name="w_neck" value="${l_neck/5}" />
-  <xacro:property name="w_upper_trunk" value="${l_upper_trunk/5}" />
-  <xacro:property name="w_lower_trunk" value="${l_lower_trunk/2}" />
-  <xacro:property name="w_upper_arm" value="${l_upper_arm/3}" />
-  <xacro:property name="w_forearm" value="${l_forearm/3}" />
-  <xacro:property name="w_hand" value="${l_hand/3}" />
-  <xacro:property name="w_thigh" value="${l_thigh/3}" />
-  <xacro:property name="w_shank" value="${l_shank/3}" />
-  <xacro:property name="w_foot" value="${l_foot/3}" />
-  <xacro:property name="cm_head" value="0.361" />
-  <xacro:property name="cm_upper_trunk" value="0.497" />
-  <xacro:property name="cm_lower_trunk" value="0.518" />
-  <xacro:property name="cm_upper_arm" value="0.427" />
-  <xacro:property name="cm_forearm" value="0.417" />
-  <xacro:property name="cm_hand" value="0.361" />
-  <xacro:property name="cm_thigh" value="0.430" />
-  <xacro:property name="cm_shank" value="0.443" />
-  <xacro:property name="cm_foot" value="0.436" />
-  <xacro:property name="d_head" value="1085.1" />
-  <xacro:property name="d_upper_trunk" value="1068.6" />
-  <xacro:property name="d_lower_trunk" value="1068.6" />
-  <xacro:property name="d_upper_arm" value="1088.0" />
-  <xacro:property name="d_forearm" value="1108.6" />
-  <xacro:property name="d_hand" value="1112.6" />
-  <xacro:property name="d_thigh" value="1068.6" />
-  <xacro:property name="d_shank" value="1100.2" />
-  <xacro:property name="d_foot" value="1089.3" />
   <xacro:include filename="$(find imu_human_pkg)/urdf/macros/spherical.xacro"/>
   <create/>

File: urdf/macros/human.gazebo.xacro (robot description, xacro)
@@ -2,24 +2,13 @@
 <robot xmlns:xacro="http://www.ros.org/wiki/xacro">
   <xacro:macro name="human_gazebo">
+    <gazebo>
+      <plugin name="gazebo_ros_control" filename="libgazebo_ros_control.so">
+        <robotNamespace>/human</robotNamespace>
+      </plugin>
+    </gazebo>
     <gazebo reference="base_link">
       <turnGravityOff>true</turnGravityOff>
       <static>true</static>
     </gazebo>
-    <!-- Wrist flex -->
-    <gazebo reference="${side}_wrist_flex_link">
-      <turnGravityOff>false</turnGravityOff>
-    </gazebo>
-    <gazebo reference="${side}_wrist_flex_joint">
-      <stopKd value="1.0" />
-      <stopKp value="1000000.0" />
-    </gazebo>
-    <!-- Wrist roll -->
-    <gazebo reference="${side}_wrist_roll_link">
-      <turnGravityOff>true</turnGravityOff>
-      <material value="PR2/RollLinks" />
-    </gazebo>
-    <gazebo reference="${side}_wrist_roll_joint">
-      <fudgeFactor value="0.5" />
-    </gazebo>
   </xacro:macro>
 </robot>

Commit message: model messed up but gazebo works. vibrating. backup

File: urdf/human/human.urdf.xacro (robot description, xacro)
@@ -3,9 +3,6 @@
   <xacro:include filename="$(find imu_human_pkg)/urdf/macros/measurements.xacro" />
   <xacro:include filename="$(find imu_human_pkg)/urdf/macros/materials.xacro" />
-  <xacro:include filename="$(find imu_human_pkg)/urdf/macros/human.gazebo.xacro" />
-  <xacro:include filename="$(find imu_human_pkg)/urdf/macros/human.transmission.xacro" />
-  <gazebo>
-    <static>true</static>
-  </gazebo>
+  <!-- <xacro:include filename="$(find imu_human_pkg)/urdf/macros/human.gazebo.xacro" />
+  <xacro:include filename="$(find imu_human_pkg)/urdf/macros/human.transmission.xacro" /> -->
   <xacro:include filename="$(find imu_human_pkg)/urdf/macros/spherical.xacro"/>
   <create/>
@@ -16,5 +13,5 @@
     <child link="base_link"/>
     <!-- <origin rpy="0.0 0.0 0.0" xyz="0 0 ${l_foot+l_shank+l_thigh+l_lower_trunk}"/> -->
-    <origin rpy="0.0 0.0 0.0" xyz="0 0 0.05"/>
+    <origin rpy="0.0 0.0 0.0" xyz="0 0 0"/>
   </joint>
   <link name="base_link">
@@ -36,18 +33,25 @@
       <mass value="${mass}"/>
       <inertia
-        ixx="${mass*(3*pow(w_upper_arm,2)+pow(l_upper_arm,2))/12}" ixy="0.0" ixz="0.0"
-        iyy="${mass*(3*pow(w_upper_arm,2)+pow(l_upper_arm,2))/12}" iyz="0.0"
-        izz="${mass*pow(w_upper_arm,2)/2}"/>
+        ixx="${2*mass*pow(0.1,2)/5}" ixy="0.0" ixz="0.0"
+        iyy="${2*mass*pow(0.1,2)/5}" iyz="0.0"
+        izz="${2*mass*pow(0.1,2)/5}"/>
     </inertial>
   </link>
-  <xacro:spherical name="joint_1" parent="base_link" child="link_01">
+  <!-- <xacro:spherical name="joint_1" parent="base_link" child="link_01">
     <origin rpy="0 0 0" xyz="0 0 0"/>
-  </xacro:spherical>
+  </xacro:spherical> -->
+  <joint name="joint_1" type="revolute">
+    <origin xyz="0 0 0.1" rpy="0 0 0" />
+    <axis xyz="0 1 0"/>
+    <parent link="base_link"/>
+    <child link="link_01"/>
+    <limit effort="1" lower="-1.57079632679" upper="1.57079632679" velocity="1"/>
+  </joint>
   <!--<xacro:cylindrical_part name="link_02" density="1" cm="1" length="5" radius="2">
     <origin rpy="0 0 0" xyz="0 0 0"/>
   </xacro:cylindrical_part>-->
   <link name="link_01">
+    <origin xyz="0 0 0" rpy="0 0 0" />
       <visual>
-        <origin xyz="0 0 ${l_upper_arm/2}" rpy="0 0 0" />
         <geometry>
           <!--<mesh filename="package://pr2_description/meshes/torso_v0/torso_lift.dae"  /> -->
@@ -57,5 +61,4 @@
       </visual>
       <collision>
-        <origin xyz="0 0 0" rpy="0 0 0"/>
         <geometry>
           <cylinder length="${l_upper_arm}" radius="${w_upper_arm}"/>
@@ -63,5 +66,4 @@
       </collision>
       <inertial>
-        <origin xyz="0 0 0" rpy="0 0 0"/>
         <mass value="${mass}"/>
         <inertia
@@ -71,3 +73,45 @@
       </inertial>
     </link>
+    <gazebo>
+        <plugin name="gazebo_ros_control" filename="libgazebo_ros_control.so">
+            <robotNamespace>/human</robotNamespace>
+            <robotParam>human_description</robotParam>
+            <controlPeriod>0.001</controlPeriod>
+            <robotSimType>gazebo_ros_control/DefaultRobotHWSim</robotSimType>
+            <!-- <legacyModeNS>true</legacyModeNS> -->
+        </plugin>
+    </gazebo>
+    <transmission name="joint_1_1_tran1">
+      <type>transmission_interface/SimpleTransmission</type>
+      <joint name="joint_1">
+        <hardwareInterface>PositionJointInterface</hardwareInterface>
+      </joint>
+      <actuator name="joint_1_1_motor1">
+        <mechanicalReduction>1</mechanicalReduction>
+      </actuator>
+    </transmission>
+<!--
+    <gazebo>
+      <plugin name="gazebo_ros_control" filename="libgazebo_ros_control.so">
+        <robotNamespace>/human</robotNamespace>
+      </plugin>
+    </gazebo>
+    <gazebo>
+      <plugin name="gazebo_ros_control" filename="libgazebo_ros_control.so">
+        <robotNamespace>/human</robotNamespace>
+        <robotSimType>gazebo_ros_control/DefaultRobotHWSim</robotSimType>
+      </plugin>
+    </gazebo> -->
+    <!-- <gazebo>
+      <plugin name="gazebo_ros_control" filename="libgazebo_ros_control.so">
+        <robotNamespace>human</robotNamespace>
+        <controlPeriod>0.001</controlPeriod>
+        <robotSimType>gazebo_ros_control/DefaultRobotHWSim</robotSimType>
+      </plugin>
+    </gazebo> -->
+    <!-- <gazebo>
+      <plugin name="gazebo_ros_control" filename="libgazebo_ros_control.so">
+        <robotNamespace>human</robotNamespace>
+      </plugin>
+    </gazebo> -->
 </robot>

File: urdf/macros/human.gazebo.xacro (robot description, xacro)
@@ -1,5 +1,4 @@
 <?xml version="1.0"?>
 <robot name="human" xmlns:xacro="http://www.ros.org/wiki/xacro">
-  <xacro:macro name="human">
     <gazebo>
       <plugin name="gazebo_ros_control" filename="libgazebo_ros_control.so">
@@ -11,4 +10,3 @@
       <static>true</static>
     </gazebo> -->
-  </xacro:macro>
 </robot>

File: urdf/macros/human.transmission.xacro (robot description, xacro)
@@ -1,5 +1,15 @@
 <?xml version="1.0"?>
 <robot name="human" xmlns:xacro="http://www.ros.org/wiki/xacro">
-  <xacro:macro name="human">
+  <transmission name="tran_1_1">
+    <type>transmission_interface/SimpleTransmission</type>
+    <joint name="joint_1_1">
+      <hardwareInterface>hardware_interface/PositionJointInterface</hardwareInterface>
+    </joint>
+    <actuator name="motor_1_1">
+      <hardwareInterface>hardware_interface/PositionJointInterface</hardwareInterface>
+      <mechanicalReduction>1</mechanicalReduction>
+    </actuator>
+  </transmission>
+<!--
     <transmission name="tran_1_1">
       <type>transmission_interface/SimpleTransmission</type>
@@ -31,5 +41,4 @@
         <mechanicalReduction>1</mechanicalReduction>
       </actuator>
-    </transmission>
-  </xacro:macro>
+    </transmission> -->
 </robot>

Commit message: only base link. building up

File: urdf/human/human.urdf.xacro (robot description, xacro)
@@ -10,4 +10,5 @@
   <link name="world"/>
   <joint name="world_joint" type="fixed">
+    <origin xyz="0 0 0.1" rpy="0 0 0" />
     <parent link="world"/>
     <child link="base_link"/>
@@ -16,6 +17,6 @@
   </joint>
   <link name="base_link">
+    <origin xyz="0 0 0.1" rpy="0 0 0" />
     <visual>
-      <origin rpy="0 0 0" xyz="0 0 0"/>
       <geometry>
         <sphere radius="0.1"/>
@@ -24,5 +25,4 @@
     </visual>
     <collision>
-      <origin xyz="0 0 0" rpy="0 0 0"/>
       <geometry>
         <sphere radius="0.1"/>
@@ -30,5 +30,4 @@
     </collision>
     <inertial>
-      <origin xyz="0 0 0" rpy="0 0 0"/>
       <mass value="${mass}"/>
       <inertia
@@ -41,5 +40,5 @@
     <origin rpy="0 0 0" xyz="0 0 0"/>
   </xacro:spherical> -->
-  <joint name="joint_1" type="revolute">
+  <!-- <joint name="joint_1" type="revolute">
     <origin xyz="0 0 0.1" rpy="0 0 0" />
     <axis xyz="0 1 0"/>
@@ -47,13 +46,12 @@
     <child link="link_01"/>
     <limit effort="1" lower="-1.57079632679" upper="1.57079632679" velocity="1"/>
-  </joint>
+  </joint> -->
   <!--<xacro:cylindrical_part name="link_02" density="1" cm="1" length="5" radius="2">
     <origin rpy="0 0 0" xyz="0 0 0"/>
   </xacro:cylindrical_part>-->
-  <link name="link_01">
+  <!-- <link name="link_01">
     <origin xyz="0 0 0" rpy="0 0 0" />
       <visual>
         <geometry>
-          <!--<mesh filename="package://pr2_description/meshes/torso_v0/torso_lift.dae"  /> -->
           <cylinder length="${l_upper_arm}" radius="${w_upper_arm}"/>
         </geometry>
@@ -72,5 +70,5 @@
           izz="${mass*pow(w_upper_arm,2)/2}"/>
       </inertial>
-    </link>
+    </link> -->
     <gazebo>
         <plugin name="gazebo_ros_control" filename="libgazebo_ros_control.so">

Commit message: ok! sth is working! controller missing

File: urdf/human/human.urdf.xacro (robot description, xacro)
@@ -8,7 +8,8 @@
   <create/>
   <xacro:property name="mass" value="${pi*l_upper_arm*pow(w_upper_arm,2)*d_upper_arm}" />
+  <xacro:property name="radius" value="0.1" />
   <link name="world"/>
   <joint name="world_joint" type="fixed">
-    <origin xyz="0 0 0.1" rpy="0 0 0" />
+    <origin xyz="0 0 ${radius}" rpy="0 0 0" />
     <parent link="world"/>
     <child link="base_link"/>
@@ -17,8 +18,7 @@
   </joint>
   <link name="base_link">
-    <origin xyz="0 0 0.1" rpy="0 0 0" />
     <visual>
       <geometry>
-        <sphere radius="0.1"/>
+        <sphere radius="${radius}"/>
       </geometry>
       <material name="white"/>
@@ -26,5 +26,5 @@
     <collision>
       <geometry>
-        <sphere radius="0.1"/>
+        <sphere radius="${radius}"/>
       </geometry>
     </collision>
@@ -32,7 +32,7 @@
       <mass value="${mass}"/>
       <inertia
-        ixx="${2*mass*pow(0.1,2)/5}" ixy="0.0" ixz="0.0"
-        iyy="${2*mass*pow(0.1,2)/5}" iyz="0.0"
-        izz="${2*mass*pow(0.1,2)/5}"/>
+        ixx="${2*mass*pow(radius,2)/5}" ixy="0.0" ixz="0.0"
+        iyy="${2*mass*pow(radius,2)/5}" iyz="0.0"
+        izz="${2*mass*pow(radius,2)/5}"/>
     </inertial>
   </link>
@@ -40,17 +40,17 @@
     <origin rpy="0 0 0" xyz="0 0 0"/>
   </xacro:spherical> -->
-  <!-- <joint name="joint_1" type="revolute">
-    <origin xyz="0 0 0.1" rpy="0 0 0" />
+  <joint name="joint_1" type="revolute">
+    <origin xyz="0 0 ${radius}" rpy="0 0 0" />
     <axis xyz="0 1 0"/>
     <parent link="base_link"/>
     <child link="link_01"/>
     <limit effort="1" lower="-1.57079632679" upper="1.57079632679" velocity="1"/>
-  </joint> -->
+  </joint>
   <!--<xacro:cylindrical_part name="link_02" density="1" cm="1" length="5" radius="2">
     <origin rpy="0 0 0" xyz="0 0 0"/>
   </xacro:cylindrical_part>-->
-  <!-- <link name="link_01">
-    <origin xyz="0 0 0" rpy="0 0 0" />
+  <link name="link_01">
       <visual>
+        <origin xyz="0 0 ${2*radius}" rpy="0 0 0" />
         <geometry>
           <cylinder length="${l_upper_arm}" radius="${w_upper_arm}"/>
@@ -59,4 +59,5 @@
       </visual>
       <collision>
+        <origin xyz="0 0 ${2*radius}" rpy="0 0 0" />
         <geometry>
           <cylinder length="${l_upper_arm}" radius="${w_upper_arm}"/>
@@ -64,4 +65,5 @@
       </collision>
       <inertial>
+        <origin xyz="0 0 ${2*radius}" rpy="0 0 0" />
         <mass value="${mass}"/>
         <inertia
@@ -70,5 +72,5 @@
           izz="${mass*pow(w_upper_arm,2)/2}"/>
       </inertial>
-    </link> -->
+    </link>
     <gazebo>
         <plugin name="gazebo_ros_control" filename="libgazebo_ros_control.so">

Commit message: gazebo and transmission xacros seperated successfully

File: urdf/human/human.urdf.xacro (robot description, xacro)
@@ -3,6 +3,6 @@
   <xacro:include filename="$(find imu_human_pkg)/urdf/macros/measurements.xacro" />
   <xacro:include filename="$(find imu_human_pkg)/urdf/macros/materials.xacro" />
-  <!-- <xacro:include filename="$(find imu_human_pkg)/urdf/macros/human.gazebo.xacro" />
-  <xacro:include filename="$(find imu_human_pkg)/urdf/macros/human.transmission.xacro" /> -->
+  <xacro:include filename="$(find imu_human_pkg)/urdf/macros/human.gazebo.xacro" />
+  <xacro:include filename="$(find imu_human_pkg)/urdf/macros/human.transmission.xacro" />
   <xacro:include filename="$(find imu_human_pkg)/urdf/macros/spherical.xacro"/>
   <create/>
@@ -73,14 +73,5 @@
       </inertial>
     </link>
-    <gazebo>
-        <plugin name="gazebo_ros_control" filename="libgazebo_ros_control.so">
-            <robotNamespace>/human</robotNamespace>
-            <robotParam>human_description</robotParam>
-            <controlPeriod>0.001</controlPeriod>
-            <robotSimType>gazebo_ros_control/DefaultRobotHWSim</robotSimType>
-            <!-- <legacyModeNS>true</legacyModeNS> -->
-        </plugin>
-    </gazebo>
-    <transmission name="joint_1_1_tran1">
+    <!-- <transmission name="joint_1_1_tran1">
       <type>transmission_interface/SimpleTransmission</type>
       <joint name="joint_1">
@@ -90,5 +81,5 @@
         <mechanicalReduction>1</mechanicalReduction>
       </actuator>
-    </transmission>
+    </transmission> -->
 <!--
     <gazebo>

File: urdf/macros/human.gazebo.xacro (robot description, xacro)
@@ -2,11 +2,11 @@
 <robot name="human" xmlns:xacro="http://www.ros.org/wiki/xacro">
     <gazebo>
-      <plugin name="gazebo_ros_control" filename="libgazebo_ros_control.so">
-        <robotNamespace>human</robotNamespace>
-      </plugin>
+        <plugin name="gazebo_ros_control" filename="libgazebo_ros_control.so">
+            <robotNamespace>/human</robotNamespace>
+            <robotParam>human_description</robotParam>
+            <controlPeriod>0.001</controlPeriod>
+            <robotSimType>gazebo_ros_control/DefaultRobotHWSim</robotSimType>
+            <!-- <legacyModeNS>true</legacyModeNS> -->
+        </plugin>
     </gazebo>
-    <!-- <gazebo reference="base_link">
-      <turnGravityOff>true</turnGravityOff>
-      <static>true</static>
-    </gazebo> -->
 </robot>

File: urdf/macros/human.transmission.xacro (robot description, xacro)
@@ -1,44 +1,12 @@
 <?xml version="1.0"?>
 <robot name="human" xmlns:xacro="http://www.ros.org/wiki/xacro">
-  <transmission name="tran_1_1">
+  <transmission name="joint_1_1_tran1">
     <type>transmission_interface/SimpleTransmission</type>
-    <joint name="joint_1_1">
+    <joint name="joint_1">
       <hardwareInterface>hardware_interface/PositionJointInterface</hardwareInterface>
     </joint>
-    <actuator name="motor_1_1">
-      <hardwareInterface>hardware_interface/PositionJointInterface</hardwareInterface>
+    <actuator name="joint_1_1_motor1">
       <mechanicalReduction>1</mechanicalReduction>
     </actuator>
   </transmission>
-<!--
-    <transmission name="tran_1_1">
-      <type>transmission_interface/SimpleTransmission</type>
-      <joint name="joint_1_1">
-        <hardwareInterface>EffortJointInterface</hardwareInterface>
-      </joint>
-      <actuator name="motor_1_1">
-        <hardwareInterface>EffortJointInterface</hardwareInterface>
-        <mechanicalReduction>1</mechanicalReduction>
-      </actuator>
-    </transmission>
-    <transmission name="tran_1_2">
-      <type>transmission_interface/SimpleTransmission</type>
-      <joint name="joint_1_2">
-        <hardwareInterface>EffortJointInterface</hardwareInterface>
-      </joint>
-      <actuator name="motor_1_2">
-        <hardwareInterface>EffortJointInterface</hardwareInterface>
-        <mechanicalReduction>1</mechanicalReduction>
-      </actuator>
-    </transmission>
-    <transmission name="tran_1_3">
-      <type>transmission_interface/SimpleTransmission</type>
-      <joint name="joint_1_3">
-        <hardwareInterface>EffortJointInterface</hardwareInterface>
-      </joint>
-      <actuator name="motor_1_3">
-        <hardwareInterface>EffortJointInterface</hardwareInterface>
-        <mechanicalReduction>1</mechanicalReduction>
-      </actuator>
-    </transmission> -->
 </robot>

Commit message: spherical joint works. plus some clean up

File: urdf/human/human.urdf.xacro (robot description, xacro)
@@ -37,8 +37,8 @@
     </inertial>
   </link>
-  <!-- <xacro:spherical name="joint_1" parent="base_link" child="link_01">
-    <origin rpy="0 0 0" xyz="0 0 0"/>
-  </xacro:spherical> -->
-  <joint name="joint_1" type="revolute">
+  <xacro:spherical name="joint_1" parent="base_link" child="link_01">
+    <origin rpy="0 0 0" xyz="0 0 ${radius}"/>
+  </xacro:spherical>
+  <!-- <joint name="joint_1" type="revolute">
     <origin xyz="0 0 ${radius}" rpy="0 0 0" />
     <axis xyz="0 1 0"/>
@@ -46,5 +46,5 @@
     <child link="link_01"/>
     <limit effort="1" lower="-1.57079632679" upper="1.57079632679" velocity="1"/>
-  </joint>
+  </joint> -->
   <!--<xacro:cylindrical_part name="link_02" density="1" cm="1" length="5" radius="2">
     <origin rpy="0 0 0" xyz="0 0 0"/>
@@ -73,36 +73,3 @@
       </inertial>
     </link>
-    <!-- <transmission name="joint_1_1_tran1">
-      <type>transmission_interface/SimpleTransmission</type>
-      <joint name="joint_1">
-        <hardwareInterface>hardware_interface/PositionJointInterface</hardwareInterface>
-      </joint>
-      <actuator name="joint_1_1_motor1">
-        <mechanicalReduction>1</mechanicalReduction>
-      </actuator>
-    </transmission> -->
-<!--
-    <gazebo>
-      <plugin name="gazebo_ros_control" filename="libgazebo_ros_control.so">
-        <robotNamespace>/human</robotNamespace>
-      </plugin>
-    </gazebo>
-    <gazebo>
-      <plugin name="gazebo_ros_control" filename="libgazebo_ros_control.so">
-        <robotNamespace>/human</robotNamespace>
-        <robotSimType>gazebo_ros_control/DefaultRobotHWSim</robotSimType>
-      </plugin>
-    </gazebo> -->
-    <!-- <gazebo>
-      <plugin name="gazebo_ros_control" filename="libgazebo_ros_control.so">
-        <robotNamespace>human</robotNamespace>
-        <controlPeriod>0.001</controlPeriod>
-        <robotSimType>gazebo_ros_control/DefaultRobotHWSim</robotSimType>
-      </plugin>
-    </gazebo> -->
-    <!-- <gazebo>
-      <plugin name="gazebo_ros_control" filename="libgazebo_ros_control.so">
-        <robotNamespace>human</robotNamespace>
-      </plugin>
-    </gazebo> -->
 </robot>

File: urdf/macros/human.transmission.xacro (robot description, xacro)
@@ -3,5 +3,5 @@
   <transmission name="joint_1_1_tran1">
     <type>transmission_interface/SimpleTransmission</type>
-    <joint name="joint_1">
+    <joint name="joint_1_1">
       <hardwareInterface>hardware_interface/PositionJointInterface</hardwareInterface>
     </joint>
@@ -10,3 +10,21 @@
     </actuator>
   </transmission>
+  <transmission name="joint_1_2_tran1">
+    <type>transmission_interface/SimpleTransmission</type>
+    <joint name="joint_1_2">
+      <hardwareInterface>hardware_interface/PositionJointInterface</hardwareInterface>
+    </joint>
+    <actuator name="joint_1_2_motor1">
+      <mechanicalReduction>1</mechanicalReduction>
+    </actuator>
+  </transmission>
+  <transmission name="joint_1_3_tran1">
+    <type>transmission_interface/SimpleTransmission</type>
+    <joint name="joint_1_3">
+      <hardwareInterface>hardware_interface/PositionJointInterface</hardwareInterface>
+    </joint>
+    <actuator name="joint_1_3_motor1">
+      <mechanicalReduction>1</mechanicalReduction>
+    </actuator>
+  </transmission>
 </robot>
