Commit message: backup. overshooting desired position.

File: urdf/human/human.urdf.xacro (robot description, xacro)
@@ -11,12 +11,13 @@
   <link name="world"/>
   <joint name="world_joint" type="fixed">
-    <origin xyz="0 0 ${radius}" rpy="0 0 0" />
+    <origin xyz="0 0 0" rpy="0 0 0" />
     <parent link="world"/>
     <child link="base_link"/>
     <!-- <origin rpy="0.0 0.0 0.0" xyz="0 0 ${l_foot+l_shank+l_thigh+l_lower_trunk}"/> -->
-    <origin rpy="0.0 0.0 0.0" xyz="0 0 0"/>
+    <origin rpy="0.0 0.0 0.0" xyz="0 0 1"/>
   </joint>
   <link name="base_link">
     <visual>
+    <origin rpy="0.0 0.0 0.0" xyz="0 0 1"/>
       <geometry>
         <sphere radius="${radius}"/>
@@ -25,4 +26,5 @@
     </visual>
     <collision>
+    <origin rpy="0.0 0.0 0.0" xyz="0 0 1"/>
       <geometry>
         <sphere radius="${radius}"/>
@@ -30,4 +32,5 @@
     </collision>
     <inertial>
+    <origin rpy="0.0 0.0 0.0" xyz="0 0 1"/>
       <mass value="${mass}"/>
       <inertia
@@ -38,5 +41,5 @@
   </link>
   <xacro:spherical name="joint_1" parent="base_link" child="link_01">
-    <origin rpy="0 0 0" xyz="0 0 ${radius}"/>
+    <origin rpy="0.0 0.0 0.0" xyz="0 0 1"/>
   </xacro:spherical>
   <!-- <joint name="joint_1" type="revolute">

File: urdf/macros/human.gazebo.xacro (robot description, xacro)
@@ -10,3 +10,7 @@
         </plugin>
     </gazebo>
+    <gazebo reference="base_link">
+        <static>true</static>
+        <turnGravityOff>true</turnGravityOff>
+    </gazebo>
 </robot>

File: urdf/macros/spherical.xacro (robot description, xacro)
@@ -3,4 +3,5 @@
 <xacro:macro name="spherical" params="name parent child *origin">
     <joint name="${name}_x" type="revolute">
+      <xacro:insert_block name="origin" />
       <axis xyz="1 0 0" />
       <limit effort="1000.0" lower="-3.14" upper="3.14" velocity="0.5"/>
@@ -39,5 +40,4 @@
     </link>
     <joint name="${name}_F" type="fixed">
-      <xacro:insert_block name="origin" />
       <parent link="${name}_virt_link_3"/>
       <child link="${child}"/>

Commit message: changed mass, P=0.1, I=1.0, controller oscilates

File: urdf/human/human.urdf.xacro (robot description, xacro)
@@ -7,5 +7,5 @@
   <xacro:include filename="$(find imu_human_pkg)/urdf/macros/spherical.xacro"/>
   <create/>
-  <xacro:property name="mass" value="${pi*l_upper_arm*pow(w_upper_arm,2)*d_upper_arm}" />
+  <xacro:property name="mass" value="${pi*l_upper_arm*pow(w_upper_arm,2)*d_upper_arm*0.0001}" />
   <xacro:property name="radius" value="0.1" />
   <link name="world"/>

Commit message: lower trunk added

File: urdf/human/human.urdf.xacro (robot description, xacro)
@@ -7,7 +7,5 @@
   <xacro:include filename="$(find imu_human_pkg)/urdf/macros/spherical.xacro"/>
   <create/>
-  <xacro:property name="mass" value="${pi*l_upper_arm*pow(w_upper_arm,2)*d_upper_arm*0.0001}" />
-  <xacro:property name="radius" value="0.1" />
-  <link name="world"/>
+    <link name="world"/>
   <joint name="world_joint" type="fixed">
     <origin xyz="0 0 0" rpy="0 0 0" />
@@ -15,32 +13,60 @@
     <child link="base_link"/>
     <!-- <origin rpy="0.0 0.0 0.0" xyz="0 0 ${l_foot+l_shank+l_thigh+l_lower_trunk}"/> -->
-    <origin rpy="0.0 0.0 0.0" xyz="0 0 1"/>
+    <origin rpy="0.0 0.0 0.0" xyz="0 0 0"/>
   </joint>
   <link name="base_link">
     <visual>
-    <origin rpy="0.0 0.0 0.0" xyz="0 0 1"/>
+    <origin rpy="0.0 0.0 0.0" xyz="0 0 ${l_foot+l_shank+l_thigh+l_lower_trunk}"/>
       <geometry>
-        <sphere radius="${radius}"/>
+        <sphere radius="${r_base_link}"/>
       </geometry>
       <material name="white"/>
     </visual>
     <collision>
-    <origin rpy="0.0 0.0 0.0" xyz="0 0 1"/>
+    <origin rpy="0.0 0.0 0.0" xyz="0 0 ${l_foot+l_shank+l_thigh+l_lower_trunk}"/>
       <geometry>
-        <sphere radius="${radius}"/>
+        <sphere radius="${r_base_link}"/>
       </geometry>
     </collision>
     <inertial>
-    <origin rpy="0.0 0.0 0.0" xyz="0 0 1"/>
-      <mass value="${mass}"/>
+    <origin rpy="0.0 0.0 0.0" xyz="0 0 ${l_foot+l_shank+l_thigh+l_lower_trunk}"/>
+      <mass value="${m_base_link}"/>
       <inertia
-        ixx="${2*mass*pow(radius,2)/5}" ixy="0.0" ixz="0.0"
-        iyy="${2*mass*pow(radius,2)/5}" iyz="0.0"
-        izz="${2*mass*pow(radius,2)/5}"/>
+        ixx="${2*m_base_link*pow(r_base_link,2)/5}" ixy="0.0" ixz="0.0"
+        iyy="${2*m_base_link*pow(r_base_link,2)/5}" iyz="0.0"
+        izz="${2*m_base_link*pow(r_base_link,2)/5}"/>
     </inertial>
   </link>
-  <xacro:spherical name="joint_1" parent="base_link" child="link_01">
+  <joint name="base_to_lower_trunk" type="fixed">
+    <origin rpy="0 0 0" xyz="0 0 ${l_foot+l_shank+l_thigh+l_lower_trunk}"/>
+    <parent link="base_link"/>
+    <child link="lower_trunk"/>
+  </joint>
+  <link name="lower_trunk">
+    <visual>
+    <origin rpy="0 0 0" xyz="0 0 0"/>
+      <geometry>
+        <cylinder length="${l_lower_trunk}" radius="${r_lower_trunk}"/>
+      </geometry>
+      <material name="white"/>
+    </visual>
+    <collision>
+    <origin rpy="0.0 0.0 0.0" xyz="0 0 0"/>
+      <geometry>
+        <cylinder length="${l_lower_trunk}" radius="${r_lower_trunk}"/>
+      </geometry>
+    </collision>
+    <inertial>
+    <origin rpy="0.0 0.0 0.0" xyz="0 0 0"/>
+      <mass value="${m_lower_trunk}"/>
+      <inertia
+        ixx="${m_lower_trunk*(3*pow(r_lower_trunk,2)+pow(l_lower_trunk,2))/12}" ixy="0.0" ixz="0.0"
+        iyy="${m_lower_trunk*(3*pow(r_lower_trunk,2)+pow(l_lower_trunk,2))/12}" iyz="0.0"
+        izz="${m_lower_trunk*pow(r_lower_trunk,2)/2}"/>
+    </inertial>
+  </link>
+  <!-- <xacro:spherical name="base_to_lower_trunk" parent="base_link" child="lower_trunk">
     <origin rpy="0.0 0.0 0.0" xyz="0 0 1"/>
-  </xacro:spherical>
+  </xacro:spherical> -->
   <!-- <joint name="joint_1" type="revolute">
     <origin xyz="0 0 ${radius}" rpy="0 0 0" />
@@ -53,5 +79,5 @@
     <origin rpy="0 0 0" xyz="0 0 0"/>
   </xacro:cylindrical_part>-->
-  <link name="link_01">
+  <!-- <link name="link_01">
       <visual>
         <origin xyz="0 0 ${2*radius}" rpy="0 0 0" />
@@ -75,4 +101,4 @@
           izz="${mass*pow(w_upper_arm,2)/2}"/>
       </inertial>
-    </link>
+    </link> -->
 </robot>

File: urdf/macros/human.transmission.xacro (robot description, xacro)
@@ -1,5 +1,5 @@
 <?xml version="1.0"?>
 <robot name="human" xmlns:xacro="http://www.ros.org/wiki/xacro">
-  <transmission name="joint_1_1_tran1">
+  <!-- <transmission name="joint_1_1_tran1">
     <type>transmission_interface/SimpleTransmission</type>
     <joint name="joint_1_x">
@@ -27,4 +27,4 @@
       <mechanicalReduction>1</mechanicalReduction>
     </actuator>
-  </transmission>
+  </transmission> -->
 </robot>

File: urdf/macros/measurements.xacro (robot description, xacro)
@@ -12,12 +12,14 @@
   <xacro:property name="l_foot" value="0.06" />
   <xacro:property name="whole_body" value="1.7268" />
-  <xacro:property name="w_neck" value="${l_neck/5}" />
-  <xacro:property name="w_upper_trunk" value="${l_upper_trunk/5}" />
-  <xacro:property name="w_lower_trunk" value="${l_lower_trunk/2}" />
-  <xacro:property name="w_upper_arm" value="${l_upper_arm/3}" />
-  <xacro:property name="w_forearm" value="${l_forearm/3}" />
+  <xacro:property name="thickness" value="0.002" />
+  <xacro:property name="r_neck" value="${l_neck/5}" />
+  <xacro:property name="r_head" value="${head/2}" />
+  <xacro:property name="r_upper_trunk" value="${l_upper_trunk/5}" />
+  <xacro:property name="r_lower_trunk" value="${l_lower_trunk/2}" />
+  <xacro:property name="r_upper_arm" value="${l_upper_arm/3}" />
+  <xacro:property name="r_forearm" value="${l_forearm/3}" />
   <xacro:property name="w_hand" value="${l_hand/3}" />
-  <xacro:property name="w_thigh" value="${l_thigh/3}" />
-  <xacro:property name="w_shank" value="${l_shank/3}" />
+  <xacro:property name="r_thigh" value="${l_thigh/3}" />
+  <xacro:property name="r_shank" value="${l_shank/3}" />
   <xacro:property name="w_foot" value="${l_foot/3}" />
   <xacro:property name="cm_head" value="0.361" />
@@ -30,4 +32,5 @@
   <xacro:property name="cm_shank" value="0.443" />
   <xacro:property name="cm_foot" value="0.436" />
+  <xacro:property name="d_neck" value="1085.1" />
   <xacro:property name="d_head" value="1085.1" />
   <xacro:property name="d_upper_trunk" value="1068.6" />
@@ -39,3 +42,17 @@
   <xacro:property name="d_shank" value="1100.2" />
   <xacro:property name="d_foot" value="1089.3" />
+  <!-- <xacro:property name="mass" value="${pi*l_upper_arm*pow(w_upper_arm,2)*d_upper_arm*0.001}" />
+  <xacro:property name="radius" value="0.1" /> -->
+  <xacro:property name="m_base_link" value="0.01" />
+  <xacro:property name="r_base_link" value="0.01" />
+  <xacro:property name="m_neck" value="${pi*l_neck*pow(r_neck,2)*d_neck*0.001}" />
+  <xacro:property name="m_head" value="${(4/3)*pi*pow(r_head,3)*0.001}" />
+  <xacro:property name="m_upper_trunk" value="${pi*l_upper_trunk*pow(r_upper_trunk,2)*d_upper_trunk*0.001}" />
+  <xacro:property name="m_lower_trunk" value="${pi*l_lower_trunk*pow(r_lower_trunk,2)*d_lower_trunk*0.001}" />
+  <xacro:property name="m_upper_arm" value="${pi*l_upper_arm*pow(r_upper_arm,2)*d_upper_arm*0.001}" />
+  <xacro:property name="m_forearm" value="${pi*l_forearm*pow(r_forearm,2)*d_forearm*0.001}" />
+  <xacro:property name="m_thigh" value="${pi*l_thigh*pow(r_thigh,2)*d_thigh*0.001}" />
+  <xacro:property name="m_shank" value="${pi*l_shank*pow(r_shank,2)*d_shank*0.001}" />
+  <xacro:property name="m_hand" value="${l_hand*w_hand*thickness*d_hand*0.001}" />
+  <xacro:property name="m_foot" value="${l_foot*w_foot*thickness*d_foot*0.001}" />
 </robot>

Commit message: left thigh added

File: urdf/human/human.urdf.xacro (robot description, xacro)
@@ -66,4 +66,32 @@
     </inertial>
   </link>
+  <joint name="lower_trunk_to_left_thigh" type="fixed">
+    <origin rpy="0 0 0" xyz="0 ${r_lower_trunk} ${-l_lower_trunk/2}"/>
+    <parent link="lower_trunk"/>
+    <child link="left_thigh"/>
+  </joint>
+  <link name="left_thigh">
+    <visual>
+    <origin rpy="0 0 0" xyz="0 0 ${-l_thigh/2}"/>
+      <geometry>
+        <cylinder length="${l_thigh}" radius="${r_thigh}"/>
+      </geometry>
+      <material name="white"/>
+    </visual>
+    <collision>
+    <origin rpy="0.0 0.0 0.0" xyz="0 0 0"/>
+      <geometry>
+        <cylinder length="${l_thigh}" radius="${r_thigh}"/>
+      </geometry>
+    </collision>
+    <inertial>
+    <origin rpy="0.0 0.0 0.0" xyz="0 0 0"/>
+      <mass value="${m_thigh}"/>
+      <inertia
+        ixx="${m_thigh*(3*pow(r_thigh,2)+pow(l_thigh,2))/12}" ixy="0.0" ixz="0.0"
+        iyy="${m_thigh*(3*pow(r_thigh,2)+pow(l_thigh,2))/12}" iyz="0.0"
+        izz="${m_thigh*pow(r_thigh,2)/2}"/>
+    </inertial>
+  </link>
   <!-- <xacro:spherical name="base_to_lower_trunk" parent="base_link" child="lower_trunk">
     <origin rpy="0.0 0.0 0.0" xyz="0 0 1"/>

File: urdf/macros/measurements.xacro (robot description, xacro)
@@ -16,5 +16,5 @@
   <xacro:property name="r_head" value="${head/2}" />
   <xacro:property name="r_upper_trunk" value="${l_upper_trunk/5}" />
-  <xacro:property name="r_lower_trunk" value="${l_lower_trunk/2}" />
+  <xacro:property name="r_lower_trunk" value="${l_lower_trunk*2}" />
   <xacro:property name="r_upper_arm" value="${l_upper_arm/3}" />
   <xacro:property name="r_forearm" value="${l_forearm/3}" />

Commit message: right thigh added

File: urdf/human/human.urdf.xacro (robot description, xacro)
@@ -67,9 +67,37 @@
   </link>
   <joint name="lower_trunk_to_left_thigh" type="fixed">
-    <origin rpy="0 0 0" xyz="0 ${r_lower_trunk} ${-l_lower_trunk/2}"/>
+    <origin rpy="0 0 0" xyz="0 ${-r_lower_trunk} ${-l_lower_trunk/2}"/>
     <parent link="lower_trunk"/>
     <child link="left_thigh"/>
   </joint>
   <link name="left_thigh">
+    <visual>
+    <origin rpy="0 0 0" xyz="0 0 ${-l_thigh/2}"/>
+      <geometry>
+        <cylinder length="${l_thigh}" radius="${r_thigh}"/>
+      </geometry>
+      <material name="white"/>
+    </visual>
+    <collision>
+    <origin rpy="0.0 0.0 0.0" xyz="0 0 0"/>
+      <geometry>
+        <cylinder length="${l_thigh}" radius="${r_thigh}"/>
+      </geometry>
+    </collision>
+    <inertial>
+    <origin rpy="0.0 0.0 0.0" xyz="0 0 0"/>
+      <mass value="${m_thigh}"/>
+      <inertia
+        ixx="${m_thigh*(3*pow(r_thigh,2)+pow(l_thigh,2))/12}" ixy="0.0" ixz="0.0"
+        iyy="${m_thigh*(3*pow(r_thigh,2)+pow(l_thigh,2))/12}" iyz="0.0"
+        izz="${m_thigh*pow(r_thigh,2)/2}"/>
+    </inertial>
+  </link>
+  <joint name="lower_trunk_to_right_thigh" type="fixed">
+    <origin rpy="0 0 0" xyz="0 ${r_lower_trunk} ${-l_lower_trunk/2}"/>
+    <parent link="lower_trunk"/>
+    <child link="right_thigh"/>
+  </joint>
+  <link name="right_thigh">
     <visual>
     <origin rpy="0 0 0" xyz="0 0 ${-l_thigh/2}"/>

Commit message: left shank added

File: urdf/human/human.urdf.xacro (robot description, xacro)
@@ -13,9 +13,9 @@
     <child link="base_link"/>
     <!-- <origin rpy="0.0 0.0 0.0" xyz="0 0 ${l_foot+l_shank+l_thigh+l_lower_trunk}"/> -->
-    <origin rpy="0.0 0.0 0.0" xyz="0 0 0"/>
+    <origin rpy="0 0 0" xyz="0 0 0"/>
   </joint>
   <link name="base_link">
     <visual>
-    <origin rpy="0.0 0.0 0.0" xyz="0 0 ${l_foot+l_shank+l_thigh+l_lower_trunk}"/>
+    <origin rpy="0 0 0" xyz="0 0 ${thickness+l_shank+l_thigh+l_lower_trunk/2}"/>
       <geometry>
         <sphere radius="${r_base_link}"/>
@@ -24,5 +24,5 @@
     </visual>
     <collision>
-    <origin rpy="0.0 0.0 0.0" xyz="0 0 ${l_foot+l_shank+l_thigh+l_lower_trunk}"/>
+    <origin rpy="0 0 0" xyz="0 0 ${thickness+l_shank+l_thigh+l_lower_trunk/2}"/>
       <geometry>
         <sphere radius="${r_base_link}"/>
@@ -30,5 +30,5 @@
     </collision>
     <inertial>
-    <origin rpy="0.0 0.0 0.0" xyz="0 0 ${l_foot+l_shank+l_thigh+l_lower_trunk}"/>
+    <origin rpy="0 0 0" xyz="0 0 ${thickness+l_shank+l_thigh+l_lower_trunk/2}"/>
       <mass value="${m_base_link}"/>
       <inertia
@@ -39,5 +39,5 @@
   </link>
   <joint name="base_to_lower_trunk" type="fixed">
-    <origin rpy="0 0 0" xyz="0 0 ${l_foot+l_shank+l_thigh+l_lower_trunk}"/>
+    <origin rpy="0 0 0" xyz="0 0 ${thickness+l_shank+l_thigh+l_lower_trunk/2}"/>
     <parent link="base_link"/>
     <child link="lower_trunk"/>
@@ -52,5 +52,5 @@
     </visual>
     <collision>
-    <origin rpy="0.0 0.0 0.0" xyz="0 0 0"/>
+    <origin rpy="0 0 0" xyz="0 0 0"/>
       <geometry>
         <cylinder length="${l_lower_trunk}" radius="${r_lower_trunk}"/>
@@ -58,5 +58,5 @@
     </collision>
     <inertial>
-    <origin rpy="0.0 0.0 0.0" xyz="0 0 0"/>
+    <origin rpy="0 0 0" xyz="0 0 0"/>
       <mass value="${m_lower_trunk}"/>
       <inertia
@@ -80,5 +80,5 @@
     </visual>
     <collision>
-    <origin rpy="0.0 0.0 0.0" xyz="0 0 0"/>
+    <origin rpy="0 0 0" xyz="0 0 ${-l_thigh/2}"/>
       <geometry>
         <cylinder length="${l_thigh}" radius="${r_thigh}"/>
@@ -86,5 +86,5 @@
     </collision>
     <inertial>
-    <origin rpy="0.0 0.0 0.0" xyz="0 0 0"/>
+    <origin rpy="0 0 0" xyz="0 0 ${-l_thigh/2}"/>
       <mass value="${m_thigh}"/>
       <inertia
@@ -108,5 +108,5 @@
     </visual>
     <collision>
-    <origin rpy="0.0 0.0 0.0" xyz="0 0 0"/>
+    <origin rpy="0 0 0" xyz="0 0 ${-l_thigh/2}"/>
       <geometry>
         <cylinder length="${l_thigh}" radius="${r_thigh}"/>
@@ -114,5 +114,5 @@
     </collision>
     <inertial>
-    <origin rpy="0.0 0.0 0.0" xyz="0 0 0"/>
+    <origin rpy="0 0 0" xyz="0 0 ${-l_thigh/2}"/>
       <mass value="${m_thigh}"/>
       <inertia
@@ -120,4 +120,32 @@
         iyy="${m_thigh*(3*pow(r_thigh,2)+pow(l_thigh,2))/12}" iyz="0.0"
         izz="${m_thigh*pow(r_thigh,2)/2}"/>
+    </inertial>
+  </link>
+  <joint name="left_thight_to_shank" type="fixed">
+    <origin rpy="0 0 0" xyz="0 0 ${-l_thigh}"/>
+    <parent link="left_thigh"/>
+    <child link="left_shank"/>
+  </joint>
+  <link name="left_shank">
+    <visual>
+    <origin rpy="0 0 0" xyz="0 0 ${-l_shank/2}"/>
+      <geometry>
+        <cylinder length="${l_shank}" radius="${r_shank}"/>
+      </geometry>
+      <material name="white"/>
+    </visual>
+    <collision>
+    <origin rpy="0.0 0.0 0.0" xyz="0 0 ${-l_shank/2}"/>
+      <geometry>
+        <cylinder length="${l_shank}" radius="${r_shank}"/>
+      </geometry>
+    </collision>
+    <inertial>
+    <origin rpy="0.0 0.0 0.0" xyz="0 0 ${-l_shank/2}"/>
+      <mass value="${m_shank}"/>
+      <inertia
+        ixx="${m_shank*(3*pow(r_shank,2)+pow(l_shank,2))/12}" ixy="0.0" ixz="0.0"
+        iyy="${m_shank*(3*pow(r_shank,2)+pow(l_shank,2))/12}" iyz="0.0"
+        izz="${m_shank*pow(r_shank,2)/2}"/>
     </inertial>
   </link>

File: urdf/macros/measurements.xacro (robot description, xacro)
@@ -20,6 +20,6 @@
   <xacro:property name="r_forearm" value="${l_forearm/3}" />
   <xacro:property name="w_hand" value="${l_hand/3}" />
-  <xacro:property name="r_thigh" value="${l_thigh/3}" />
-  <xacro:property name="r_shank" value="${l_shank/3}" />
+  <xacro:property name="r_thigh" value="${l_thigh/4}" />
+  <xacro:property name="r_shank" value="${l_shank/5}" />
   <xacro:property name="w_foot" value="${l_foot/3}" />
   <xacro:property name="cm_head" value="0.361" />

Commit message: left leg and foot completed

File: urdf/human/human.urdf.xacro (robot description, xacro)
@@ -148,4 +148,32 @@
         iyy="${m_shank*(3*pow(r_shank,2)+pow(l_shank,2))/12}" iyz="0.0"
         izz="${m_shank*pow(r_shank,2)/2}"/>
+    </inertial>
+  </link>
+  <joint name="left_shank_to_foot" type="fixed">
+    <origin rpy="0 0 0" xyz="0 0 ${-l_shank}"/>
+    <parent link="left_shank"/>
+    <child link="left_foot"/>
+  </joint>
+  <link name="left_foot">
+    <visual>
+    <origin rpy="0 0 0" xyz="${r_shank/2} 0 ${-thickness/2}"/>
+      <geometry>
+        <box size="${l_foot} ${w_foot} ${thickness}"/>
+      </geometry>
+      <material name="white"/>
+    </visual>
+    <collision>
+    <origin rpy="0.0 0.0 0.0" xyz="0 0 ${-thickness/2}"/>
+      <geometry>
+        <box size="${l_foot} ${w_foot} ${thickness}"/>
+      </geometry>
+    </collision>
+    <inertial>
+    <origin rpy="0.0 0.0 0.0" xyz="0 0 ${-l_shank/2}"/>
+      <mass value="${m_hand}"/>
+      <inertia
+        ixx="${m_hand*(pow(thickness,2) + pow(w_hand,2))/12}" ixy="0.0" ixz="0.0"
+        iyy="${m_hand*(pow(l_hand,2) + pow(thickness,2))/12}" iyz="0.0"
+        izz="${m_hand*(pow(l_hand,2) + pow(w_hand,2))/12}"/>
     </inertial>
   </link>

File: urdf/macros/measurements.xacro (robot description, xacro)
@@ -10,17 +10,17 @@
   <xacro:property name="l_thigh" value="0.449" />
   <xacro:property name="l_shank" value="0.429" />
-  <xacro:property name="l_foot" value="0.06" />
+  <xacro:property name="l_foot" value="${w_foot*4}" />
   <xacro:property name="whole_body" value="1.7268" />
-  <xacro:property name="thickness" value="0.002" />
+  <xacro:property name="thickness" value="0.02" />
   <xacro:property name="r_neck" value="${l_neck/5}" />
   <xacro:property name="r_head" value="${head/2}" />
   <xacro:property name="r_upper_trunk" value="${l_upper_trunk/5}" />
-  <xacro:property name="r_lower_trunk" value="${l_lower_trunk*2}" />
+  <xacro:property name="r_lower_trunk" value="${l_lower_trunk*1.25}" />
   <xacro:property name="r_upper_arm" value="${l_upper_arm/3}" />
   <xacro:property name="r_forearm" value="${l_forearm/3}" />
   <xacro:property name="w_hand" value="${l_hand/3}" />
-  <xacro:property name="r_thigh" value="${l_thigh/4}" />
-  <xacro:property name="r_shank" value="${l_shank/5}" />
-  <xacro:property name="w_foot" value="${l_foot/3}" />
+  <xacro:property name="r_thigh" value="${l_thigh/5}" />
+  <xacro:property name="r_shank" value="${l_shank/6}" />
+  <xacro:property name="w_foot" value="0.06" />
   <xacro:property name="cm_head" value="0.361" />
   <xacro:property name="cm_upper_trunk" value="0.497" />

Commit message: right leg and foot completed

File: urdf/human/human.urdf.xacro (robot description, xacro)
@@ -7,5 +7,5 @@
   <xacro:include filename="$(find imu_human_pkg)/urdf/macros/spherical.xacro"/>
   <create/>
-    <link name="world"/>
+  <link name="world"/>
   <joint name="world_joint" type="fixed">
     <origin xyz="0 0 0" rpy="0 0 0" />
@@ -156,4 +156,60 @@
   </joint>
   <link name="left_foot">
+    <visual>
+    <origin rpy="0 0 0" xyz="${r_shank/2} 0 ${-thickness/2}"/>
+      <geometry>
+        <box size="${l_foot} ${w_foot} ${thickness}"/>
+      </geometry>
+      <material name="white"/>
+    </visual>
+    <collision>
+    <origin rpy="0.0 0.0 0.0" xyz="0 0 ${-thickness/2}"/>
+      <geometry>
+        <box size="${l_foot} ${w_foot} ${thickness}"/>
+      </geometry>
+    </collision>
+    <inertial>
+    <origin rpy="0.0 0.0 0.0" xyz="0 0 ${-l_shank/2}"/>
+      <mass value="${m_hand}"/>
+      <inertia
+        ixx="${m_hand*(pow(thickness,2) + pow(w_hand,2))/12}" ixy="0.0" ixz="0.0"
+        iyy="${m_hand*(pow(l_hand,2) + pow(thickness,2))/12}" iyz="0.0"
+        izz="${m_hand*(pow(l_hand,2) + pow(w_hand,2))/12}"/>
+    </inertial>
+  </link>
+    <joint name="right_thight_to_shank" type="fixed">
+    <origin rpy="0 0 0" xyz="0 0 ${-l_thigh}"/>
+    <parent link="right_thigh"/>
+    <child link="right_shank"/>
+  </joint>
+  <link name="right_shank">
+    <visual>
+    <origin rpy="0 0 0" xyz="0 0 ${-l_shank/2}"/>
+      <geometry>
+        <cylinder length="${l_shank}" radius="${r_shank}"/>
+      </geometry>
+      <material name="white"/>
+    </visual>
+    <collision>
+    <origin rpy="0.0 0.0 0.0" xyz="0 0 ${-l_shank/2}"/>
+      <geometry>
+        <cylinder length="${l_shank}" radius="${r_shank}"/>
+      </geometry>
+    </collision>
+    <inertial>
+    <origin rpy="0.0 0.0 0.0" xyz="0 0 ${-l_shank/2}"/>
+      <mass value="${m_shank}"/>
+      <inertia
+        ixx="${m_shank*(3*pow(r_shank,2)+pow(l_shank,2))/12}" ixy="0.0" ixz="0.0"
+        iyy="${m_shank*(3*pow(r_shank,2)+pow(l_shank,2))/12}" iyz="0.0"
+        izz="${m_shank*pow(r_shank,2)/2}"/>
+    </inertial>
+  </link>
+  <joint name="right_shank_to_foot" type="fixed">
+    <origin rpy="0 0 0" xyz="0 0 ${-l_shank}"/>
+    <parent link="right_shank"/>
+    <child link="right_foot"/>
+  </joint>
+  <link name="right_foot">
     <visual>
     <origin rpy="0 0 0" xyz="${r_shank/2} 0 ${-thickness/2}"/>
