Commit message: human lower body is in xacro

File: urdf/human/human.urdf.xacro (robot description, xacro)
@@ -6,4 +6,5 @@
   <xacro:include filename="$(find imu_human_pkg)/urdf/macros/human.transmission.xacro" />
   <xacro:include filename="$(find imu_human_pkg)/urdf/macros/spherical.xacro"/>
+  <xacro:include filename="$(find imu_human_pkg)/urdf/human/human_lower.xacro"/>
   <create/>
   <link name="world"/>
@@ -38,200 +39,5 @@
     </inertial>
   </link>
-  <joint name="base_to_lower_trunk" type="fixed">
-    <origin rpy="0 0 0" xyz="0 0 ${thickness+l_shank+l_thigh+l_lower_trunk/2}"/>
-    <parent link="base_link"/>
-    <child link="lower_trunk"/>
-  </joint>
-  <link name="lower_trunk">
-    <visual>
-    <origin rpy="0 0 0" xyz="0 0 0"/>
-      <geometry>
-        <cylinder length="${l_lower_trunk}" radius="${r_lower_trunk}"/>
-      </geometry>
-      <material name="white"/>
-    </visual>
-    <collision>
-    <origin rpy="0 0 0" xyz="0 0 0"/>
-      <geometry>
-        <cylinder length="${l_lower_trunk}" radius="${r_lower_trunk}"/>
-      </geometry>
-    </collision>
-    <inertial>
-    <origin rpy="0 0 0" xyz="0 0 0"/>
-      <mass value="${m_lower_trunk}"/>
-      <inertia
-        ixx="${m_lower_trunk*(3*pow(r_lower_trunk,2)+pow(l_lower_trunk,2))/12}" ixy="0.0" ixz="0.0"
-        iyy="${m_lower_trunk*(3*pow(r_lower_trunk,2)+pow(l_lower_trunk,2))/12}" iyz="0.0"
-        izz="${m_lower_trunk*pow(r_lower_trunk,2)/2}"/>
-    </inertial>
-  </link>
-  <joint name="lower_trunk_to_left_thigh" type="fixed">
-    <origin rpy="0 0 0" xyz="0 ${-r_lower_trunk} ${-l_lower_trunk/2}"/>
-    <parent link="lower_trunk"/>
-    <child link="left_thigh"/>
-  </joint>
-  <link name="left_thigh">
-    <visual>
-    <origin rpy="0 0 0" xyz="0 0 ${-l_thigh/2}"/>
-      <geometry>
-        <cylinder length="${l_thigh}" radius="${r_thigh}"/>
-      </geometry>
-      <material name="white"/>
-    </visual>
-    <collision>
-    <origin rpy="0 0 0" xyz="0 0 ${-l_thigh/2}"/>
-      <geometry>
-        <cylinder length="${l_thigh}" radius="${r_thigh}"/>
-      </geometry>
-    </collision>
-    <inertial>
-    <origin rpy="0 0 0" xyz="0 0 ${-l_thigh/2}"/>
-      <mass value="${m_thigh}"/>
-      <inertia
-        ixx="${m_thigh*(3*pow(r_thigh,2)+pow(l_thigh,2))/12}" ixy="0.0" ixz="0.0"
-        iyy="${m_thigh*(3*pow(r_thigh,2)+pow(l_thigh,2))/12}" iyz="0.0"
-        izz="${m_thigh*pow(r_thigh,2)/2}"/>
-    </inertial>
-  </link>
-  <joint name="lower_trunk_to_right_thigh" type="fixed">
-    <origin rpy="0 0 0" xyz="0 ${r_lower_trunk} ${-l_lower_trunk/2}"/>
-    <parent link="lower_trunk"/>
-    <child link="right_thigh"/>
-  </joint>
-  <link name="right_thigh">
-    <visual>
-    <origin rpy="0 0 0" xyz="0 0 ${-l_thigh/2}"/>
-      <geometry>
-        <cylinder length="${l_thigh}" radius="${r_thigh}"/>
-      </geometry>
-      <material name="white"/>
-    </visual>
-    <collision>
-    <origin rpy="0 0 0" xyz="0 0 ${-l_thigh/2}"/>
-      <geometry>
-        <cylinder length="${l_thigh}" radius="${r_thigh}"/>
-      </geometry>
-    </collision>
-    <inertial>
-    <origin rpy="0 0 0" xyz="0 0 ${-l_thigh/2}"/>
-      <mass value="${m_thigh}"/>
-      <inertia
-        ixx="${m_thigh*(3*pow(r_thigh,2)+pow(l_thigh,2))/12}" ixy="0.0" ixz="0.0"
-        iyy="${m_thigh*(3*pow(r_thigh,2)+pow(l_thigh,2))/12}" iyz="0.0"
-        izz="${m_thigh*pow(r_thigh,2)/2}"/>
-    </inertial>
-  </link>
-  <joint name="left_thight_to_shank" type="fixed">
-    <origin rpy="0 0 0" xyz="0 0 ${-l_thigh}"/>
-    <parent link="left_thigh"/>
-    <child link="left_shank"/>
-  </joint>
-  <link name="left_shank">
-    <visual>
-    <origin rpy="0 0 0" xyz="0 0 ${-l_shank/2}"/>
-      <geometry>
-        <cylinder length="${l_shank}" radius="${r_shank}"/>
-      </geometry>
-      <material name="white"/>
-    </visual>
-    <collision>
-    <origin rpy="0.0 0.0 0.0" xyz="0 0 ${-l_shank/2}"/>
-      <geometry>
-        <cylinder length="${l_shank}" radius="${r_shank}"/>
-      </geometry>
-    </collision>
-    <inertial>
-    <origin rpy="0.0 0.0 0.0" xyz="0 0 ${-l_shank/2}"/>
-      <mass value="${m_shank}"/>
-      <inertia
-        ixx="${m_shank*(3*pow(r_shank,2)+pow(l_shank,2))/12}" ixy="0.0" ixz="0.0"
-        iyy="${m_shank*(3*pow(r_shank,2)+pow(l_shank,2))/12}" iyz="0.0"
-        izz="${m_shank*pow(r_shank,2)/2}"/>
-    </inertial>
-  </link>
-  <joint name="left_shank_to_foot" type="fixed">
-    <origin rpy="0 0 0" xyz="0 0 ${-l_shank}"/>
-    <parent link="left_shank"/>
-    <child link="left_foot"/>
-  </joint>
-  <link name="left_foot">
-    <visual>
-    <origin rpy="0 0 0" xyz="${r_shank/2} 0 ${-thickness/2}"/>
-      <geometry>
-        <box size="${l_foot} ${w_foot} ${thickness}"/>
-      </geometry>
-      <material name="white"/>
-    </visual>
-    <collision>
-    <origin rpy="0.0 0.0 0.0" xyz="0 0 ${-thickness/2}"/>
-      <geometry>
-        <box size="${l_foot} ${w_foot} ${thickness}"/>
-      </geometry>
-    </collision>
-    <inertial>
-    <origin rpy="0.0 0.0 0.0" xyz="0 0 ${-l_shank/2}"/>
-      <mass value="${m_hand}"/>
-      <inertia
-        ixx="${m_hand*(pow(thickness,2) + pow(w_hand,2))/12}" ixy="0.0" ixz="0.0"
-        iyy="${m_hand*(pow(l_hand,2) + pow(thickness,2))/12}" iyz="0.0"
-        izz="${m_hand*(pow(l_hand,2) + pow(w_hand,2))/12}"/>
-    </inertial>
-  </link>
-    <joint name="right_thight_to_shank" type="fixed">
-    <origin rpy="0 0 0" xyz="0 0 ${-l_thigh}"/>
-    <parent link="right_thigh"/>
-    <child link="right_shank"/>
-  </joint>
-  <link name="right_shank">
-    <visual>
-    <origin rpy="0 0 0" xyz="0 0 ${-l_shank/2}"/>
-      <geometry>
-        <cylinder length="${l_shank}" radius="${r_shank}"/>
-      </geometry>
-      <material name="white"/>
-    </visual>
-    <collision>
-    <origin rpy="0.0 0.0 0.0" xyz="0 0 ${-l_shank/2}"/>
-      <geometry>
-        <cylinder length="${l_shank}" radius="${r_shank}"/>
-      </geometry>
-    </collision>
-    <inertial>
-    <origin rpy="0.0 0.0 0.0" xyz="0 0 ${-l_shank/2}"/>
-      <mass value="${m_shank}"/>
-      <inertia
-        ixx="${m_shank*(3*pow(r_shank,2)+pow(l_shank,2))/12}" ixy="0.0" ixz="0.0"
-        iyy="${m_shank*(3*pow(r_shank,2)+pow(l_shank,2))/12}" iyz="0.0"
-        izz="${m_shank*pow(r_shank,2)/2}"/>
-    </inertial>
-  </link>
-  <joint name="right_shank_to_foot" type="fixed">
-    <origin rpy="0 0 0" xyz="0 0 ${-l_shank}"/>
-    <parent link="right_shank"/>
-    <child link="right_foot"/>
-  </joint>
-  <link name="right_foot">
-    <visual>
-    <origin rpy="0 0 0" xyz="${r_shank/2} 0 ${-thickness/2}"/>
-      <geometry>
-        <box size="${l_foot} ${w_foot} ${thickness}"/>
-      </geometry>
-      <material name="white"/>
-    </visual>
-    <collision>
-    <origin rpy="0.0 0.0 0.0" xyz="0 0 ${-thickness/2}"/>
-      <geometry>
-        <box size="${l_foot} ${w_foot} ${thickness}"/>
-      </geometry>
-    </collision>
-    <inertial>
-    <origin rpy="0.0 0.0 0.0" xyz="0 0 ${-l_shank/2}"/>
-      <mass value="${m_hand}"/>
-      <inertia
-        ixx="${m_hand*(pow(thickness,2) + pow(w_hand,2))/12}" ixy="0.0" ixz="0.0"
-        iyy="${m_hand*(pow(l_hand,2) + pow(thickness,2))/12}" iyz="0.0"
-        izz="${m_hand*(pow(l_hand,2) + pow(w_hand,2))/12}"/>
-    </inertial>
-  </link>
+  <xacro:human_lower />
   <!-- <xacro:spherical name="base_to_lower_trunk" parent="base_link" child="lower_trunk">
     <origin rpy="0.0 0.0 0.0" xyz="0 0 1"/>

Commit message: tiny fix on feet

File: urdf/human/human.urdf.xacro (robot description, xacro)
@@ -7,4 +7,5 @@
   <xacro:include filename="$(find imu_human_pkg)/urdf/macros/spherical.xacro"/>
   <xacro:include filename="$(find imu_human_pkg)/urdf/human/human_lower.xacro"/>
+  <!-- <xacro:include filename="$(find imu_human_pkg)/urdf/human/human_upper.xacro"/> -->
   <create/>
   <link name="world"/>
@@ -13,5 +14,4 @@
     <parent link="world"/>
     <child link="base_link"/>
-    <!-- <origin rpy="0.0 0.0 0.0" xyz="0 0 ${l_foot+l_shank+l_thigh+l_lower_trunk}"/> -->
     <origin rpy="0 0 0" xyz="0 0 0"/>
   </joint>
@@ -39,40 +39,5 @@
     </inertial>
   </link>
-  <xacro:human_lower />
-  <!-- <xacro:spherical name="base_to_lower_trunk" parent="base_link" child="lower_trunk">
-    <origin rpy="0.0 0.0 0.0" xyz="0 0 1"/>
-  </xacro:spherical> -->
-  <!-- <joint name="joint_1" type="revolute">
-    <origin xyz="0 0 ${radius}" rpy="0 0 0" />
-    <axis xyz="0 1 0"/>
-    <parent link="base_link"/>
-    <child link="link_01"/>
-    <limit effort="1" lower="-1.57079632679" upper="1.57079632679" velocity="1"/>
-  </joint> -->
-  <!--<xacro:cylindrical_part name="link_02" density="1" cm="1" length="5" radius="2">
-    <origin rpy="0 0 0" xyz="0 0 0"/>
-  </xacro:cylindrical_part>-->
-  <!-- <link name="link_01">
-      <visual>
-        <origin xyz="0 0 ${2*radius}" rpy="0 0 0" />
-        <geometry>
-          <cylinder length="${l_upper_arm}" radius="${w_upper_arm}"/>
-        </geometry>
-        <material name="blue" />
-      </visual>
-      <collision>
-        <origin xyz="0 0 ${2*radius}" rpy="0 0 0" />
-        <geometry>
-          <cylinder length="${l_upper_arm}" radius="${w_upper_arm}"/>
-        </geometry>
-      </collision>
-      <inertial>
-        <origin xyz="0 0 ${2*radius}" rpy="0 0 0" />
-        <mass value="${mass}"/>
-        <inertia
-          ixx="${mass*(3*pow(w_upper_arm,2)+pow(l_upper_arm,2))/12}" ixy="0.0" ixz="0.0"
-          iyy="${mass*(3*pow(w_upper_arm,2)+pow(l_upper_arm,2))/12}" iyz="0.0"
-          izz="${mass*pow(w_upper_arm,2)/2}"/>
-      </inertial>
-    </link> -->
+  <xacro:human_lower/>
+  <!-- <xacro:human_upper/> -->
 </robot>

File: urdf/human/human_lower.xacro (robot description, xacro)
@@ -135,9 +135,9 @@
         <inertial>
         <origin rpy="0.0 0.0 0.0" xyz="0 0 ${-l_shank/2}"/>
-        <mass value="${m_hand}"/>
-        <inertia
-            ixx="${m_hand*(pow(thickness,2) + pow(w_hand,2))/12}" ixy="0.0" ixz="0.0"
-            iyy="${m_hand*(pow(l_hand,2) + pow(thickness,2))/12}" iyz="0.0"
-            izz="${m_hand*(pow(l_hand,2) + pow(w_hand,2))/12}"/>
+        <mass value="${m_foot}"/>
+        <inertia
+            ixx="${m_foot*(pow(thickness,2) + pow(w_foot,2))/12}" ixy="0.0" ixz="0.0"
+            iyy="${m_foot*(pow(l_foot,2) + pow(thickness,2))/12}" iyz="0.0"
+            izz="${m_foot*(pow(l_foot,2) + pow(w_foot,2))/12}"/>
         </inertial>
     </link>
@@ -191,9 +191,9 @@
         <inertial>
         <origin rpy="0.0 0.0 0.0" xyz="0 0 ${-l_shank/2}"/>
-        <mass value="${m_hand}"/>
-        <inertia
-            ixx="${m_hand*(pow(thickness,2) + pow(w_hand,2))/12}" ixy="0.0" ixz="0.0"
-            iyy="${m_hand*(pow(l_hand,2) + pow(thickness,2))/12}" iyz="0.0"
-            izz="${m_hand*(pow(l_hand,2) + pow(w_hand,2))/12}"/>
+        <mass value="${m_foot}"/>
+        <inertia
+            ixx="${m_foot*(pow(thickness,2) + pow(w_foot,2))/12}" ixy="0.0" ixz="0.0"
+            iyy="${m_foot*(pow(l_foot,2) + pow(thickness,2))/12}" iyz="0.0"
+            izz="${m_foot*(pow(l_foot,2) + pow(w_foot,2))/12}"/>
         </inertial>
     </link>

Commit message: upper thunk added

File: urdf/human/human.urdf.xacro (robot description, xacro)
@@ -7,5 +7,5 @@
   <xacro:include filename="$(find imu_human_pkg)/urdf/macros/spherical.xacro"/>
   <xacro:include filename="$(find imu_human_pkg)/urdf/human/human_lower.xacro"/>
-  <!-- <xacro:include filename="$(find imu_human_pkg)/urdf/human/human_upper.xacro"/> -->
+  <xacro:include filename="$(find imu_human_pkg)/urdf/human/human_upper.xacro"/>
   <create/>
   <link name="world"/>
@@ -40,4 +40,4 @@
   </link>
   <xacro:human_lower/>
-  <!-- <xacro:human_upper/> -->
+  <xacro:human_upper/>
 </robot>

File: urdf/macros/measurements.xacro (robot description, xacro)
@@ -15,5 +15,5 @@
   <xacro:property name="r_neck" value="${l_neck/5}" />
   <xacro:property name="r_head" value="${head/2}" />
-  <xacro:property name="r_upper_trunk" value="${l_upper_trunk/5}" />
+  <xacro:property name="r_upper_trunk" value="${l_upper_trunk/2}" />
   <xacro:property name="r_lower_trunk" value="${l_lower_trunk*1.25}" />
   <xacro:property name="r_upper_arm" value="${l_upper_arm/3}" />

Commit message: tiny addition to initial direction

File: urdf/human/human.urdf.xacro (robot description, xacro)
@@ -11,4 +11,5 @@
   <link name="world"/>
   <joint name="world_joint" type="fixed">
+    <!-- <origin xyz="0 0 0" rpy="0 0 ${pi/2}" /> -->
     <origin xyz="0 0 0" rpy="0 0 0" />
     <parent link="world"/>
