Commit message: left elbow added as 3 dof

File: urdf/human/human_lower.xacro (robot description, xacro)
@@ -31,5 +31,5 @@
     </link>
     <joint name="lower_trunk_to_left_thigh" type="fixed">
-        <origin rpy="0 0 0" xyz="0 ${-r_lower_trunk} ${-l_lower_trunk/2}"/>
+        <origin rpy="0 0 0" xyz="0 ${-r_lower_trunk/2} ${-l_lower_trunk/2}"/>
         <parent link="lower_trunk"/>
         <child link="left_thigh"/>
@@ -59,5 +59,5 @@
     </link>
     <joint name="lower_trunk_to_right_thigh" type="fixed">
-        <origin rpy="0 0 0" xyz="0 ${r_lower_trunk} ${-l_lower_trunk/2}"/>
+        <origin rpy="0 0 0" xyz="0 ${r_lower_trunk/2} ${-l_lower_trunk/2}"/>
         <parent link="lower_trunk"/>
         <child link="right_thigh"/>

File: urdf/human/human_upper.xacro (robot description, xacro)
@@ -80,4 +80,30 @@
         </inertial>
     </link>
+    <xacro:spherical name="left_elbow" parent="left_upper_arm" child="left_forearm" x="0" y="1" z="-1">
+        <origin rpy="0 0 0" xyz="0 0 ${-l_upper_arm}"/>
+    </xacro:spherical>
+    <link name="left_forearm">
+        <visual>
+        <origin rpy="0 0 0" xyz="0 0 ${-l_forearm/2}"/>
+        <geometry>
+            <cylinder length="${l_forearm}" radius="${r_forearm}"/>
+        </geometry>
+        <material name="orange"/>
+        </visual>
+        <collision>
+        <origin rpy="0 0 0" xyz="0 0 ${-l_forearm/2}"/>
+        <geometry>
+            <cylinder length="${l_forearm}" radius="${r_forearm}"/>
+        </geometry>
+        </collision>
+        <inertial>
+        <origin rpy="0 0 0" xyz="0 0 ${-l_forearm/2}"/>
+        <mass value="${m_forearm}"/>
+        <inertia
+            ixx="${m_forearm*(3*pow(r_forearm,2)+pow(l_forearm,2))/12}" ixy="0.0" ixz="0.0"
+            iyy="${m_forearm*(3*pow(r_forearm,2)+pow(l_forearm,2))/12}" iyz="0.0"
+            izz="${m_forearm*pow(r_upper_arm,2)/2}"/>
+        </inertial>
+    </link>
 </xacro:macro>
 </robot>

File: urdf/macros/human.transmission.xacro (robot description, xacro)
@@ -82,28 +82,28 @@
     </actuator>
   </transmission>
-  <!-- <transmission name="joint_1_1_tran1">
+  <!-- <transmission name="left_elbow_y_trans">
     <type>transmission_interface/SimpleTransmission</type>
-    <joint name="joint_1_x">
+    <joint name="left_elbow_y">
       <hardwareInterface>hardware_interface/PositionJointInterface</hardwareInterface>
     </joint>
-    <actuator name="joint_1_1_motor1">
+    <actuator name="left_elbow_y_motor">
       <mechanicalReduction>1</mechanicalReduction>
     </actuator>
   </transmission>
-  <transmission name="joint_1_2_tran1">
+  <transmission name="left_elbow_x_trans">
     <type>transmission_interface/SimpleTransmission</type>
-    <joint name="joint_1_y">
+    <joint name="left_elbow_x">
       <hardwareInterface>hardware_interface/PositionJointInterface</hardwareInterface>
     </joint>
-    <actuator name="joint_1_2_motor1">
+    <actuator name="left_elbow_x_motor">
       <mechanicalReduction>1</mechanicalReduction>
     </actuator>
   </transmission>
-  <transmission name="joint_1_3_tran1">
+  <transmission name="left_elbow_z_trans">
     <type>transmission_interface/SimpleTransmission</type>
-    <joint name="joint_1_z">
+    <joint name="left_elbow_z">
       <hardwareInterface>hardware_interface/PositionJointInterface</hardwareInterface>
     </joint>
-    <actuator name="joint_1_3_motor1">
+    <actuator name="left_elbow_z_motor">
       <mechanicalReduction>1</mechanicalReduction>
     </actuator>

File: urdf/macros/materials.xacro (robot description, xacro)
@@ -10,3 +10,9 @@
     <color rgba="1 1 1 1"/>
   </material>
+  <material name="green">
+    <color rgba="0 0.8 0 0.8"/>
+  </material>
+  <material name="orange">
+    <color rgba="1 0.6 0 0.8"/>
+  </material>
 </robot>

File: urdf/macros/measurements.xacro (robot description, xacro)
@@ -3,7 +3,10 @@
   <xacro:property name="l_neck" value="0.053" />
   <xacro:property name="head" value="0.212-${neck}" />
-  <xacro:property name="l_upper_trunk" value="0.410" />
-  <xacro:property name="l_lower_trunk" value="0.135" />
-  <xacro:property name="l_upper_arm" value="0.65" />
+  <!-- <xacro:property name="l_upper_trunk" value="0.410" /> -->
+  <xacro:property name="l_upper_trunk" value="0.510" />
+  <!-- <xacro:property name="l_lower_trunk" value="0.135" /> -->
+  <xacro:property name="l_lower_trunk" value="0.235" />
+  <!-- <xacro:property name="l_upper_arm" value="0.65" /> -->
+  <xacro:property name="l_upper_arm" value="0.5" />
   <xacro:property name="l_forearm" value="0.299" />
   <xacro:property name="l_hand" value="0.203" />
@@ -15,11 +18,11 @@
   <xacro:property name="r_neck" value="${l_neck/5}" />
   <xacro:property name="r_head" value="${head/2}" />
-  <xacro:property name="r_upper_trunk" value="${l_upper_trunk/2}" />
+  <xacro:property name="r_upper_trunk" value="${l_upper_trunk/1.5}" />
   <xacro:property name="r_lower_trunk" value="${l_lower_trunk*1.25}" />
   <xacro:property name="r_upper_arm" value="${l_upper_arm/6}" />
   <xacro:property name="r_forearm" value="${l_forearm/7}" />
   <xacro:property name="w_hand" value="${l_hand/3}" />
-  <xacro:property name="r_thigh" value="${l_thigh/5}" />
-  <xacro:property name="r_shank" value="${l_shank/6}" />
+  <xacro:property name="r_thigh" value="${l_thigh/4}" />
+  <xacro:property name="r_shank" value="${l_shank/5}" />
   <xacro:property name="w_foot" value="0.06" />
   <xacro:property name="cm_head" value="0.361" />

Commit message: model measurements update

File: urdf/human/human_lower.xacro (robot description, xacro)
@@ -100,11 +100,11 @@
         </visual>
         <collision>
-        <origin rpy="0.0 0.0 0.0" xyz="0 0 ${-l_shank/2}"/>
-        <geometry>
-            <cylinder length="${l_shank}" radius="${r_shank}"/>
-        </geometry>
-        </collision>
-        <inertial>
-        <origin rpy="0.0 0.0 0.0" xyz="0 0 ${-l_shank/2}"/>
+        <origin rpy="0 0 0" xyz="0 0 ${-l_shank/2}"/>
+        <geometry>
+            <cylinder length="${l_shank}" radius="${r_shank}"/>
+        </geometry>
+        </collision>
+        <inertial>
+        <origin rpy="0 0 0" xyz="0 0 ${-l_shank/2}"/>
         <mass value="${m_shank}"/>
         <inertia
@@ -128,11 +128,11 @@
         </visual>
         <collision>
-        <origin rpy="0.0 0.0 0.0" xyz="0 0 ${-thickness/2}"/>
-        <geometry>
-            <box size="${l_foot} ${w_foot} ${thickness}"/>
-        </geometry>
-        </collision>
-        <inertial>
-        <origin rpy="0.0 0.0 0.0" xyz="0 0 ${-l_shank/2}"/>
+        <origin rpy="0 0 0" xyz="0 0 ${-thickness/2}"/>
+        <geometry>
+            <box size="${l_foot} ${w_foot} ${thickness}"/>
+        </geometry>
+        </collision>
+        <inertial>
+        <origin rpy="0 0 0" xyz="0 0 ${-l_shank/2}"/>
         <mass value="${m_foot}"/>
         <inertia
@@ -156,11 +156,11 @@
         </visual>
         <collision>
-        <origin rpy="0.0 0.0 0.0" xyz="0 0 ${-l_shank/2}"/>
-        <geometry>
-            <cylinder length="${l_shank}" radius="${r_shank}"/>
-        </geometry>
-        </collision>
-        <inertial>
-        <origin rpy="0.0 0.0 0.0" xyz="0 0 ${-l_shank/2}"/>
+        <origin rpy="0 0 0" xyz="0 0 ${-l_shank/2}"/>
+        <geometry>
+            <cylinder length="${l_shank}" radius="${r_shank}"/>
+        </geometry>
+        </collision>
+        <inertial>
+        <origin rpy="0 0 0" xyz="0 0 ${-l_shank/2}"/>
         <mass value="${m_shank}"/>
         <inertia
@@ -184,11 +184,11 @@
         </visual>
         <collision>
-        <origin rpy="0.0 0.0 0.0" xyz="0 0 ${-thickness/2}"/>
-        <geometry>
-            <box size="${l_foot} ${w_foot} ${thickness}"/>
-        </geometry>
-        </collision>
-        <inertial>
-        <origin rpy="0.0 0.0 0.0" xyz="0 0 ${-l_shank/2}"/>
+        <origin rpy="0 0 0" xyz="0 0 ${-thickness/2}"/>
+        <geometry>
+            <box size="${l_foot} ${w_foot} ${thickness}"/>
+        </geometry>
+        </collision>
+        <inertial>
+        <origin rpy="0 0 0" xyz="0 0 ${-l_shank/2}"/>
         <mass value="${m_foot}"/>
         <inertia

File: urdf/human/human_upper.xacro (robot description, xacro)
@@ -152,5 +152,5 @@
         </inertial> -->
     </link>
-    <joint name="joint_neck" type="fixed">
+    <joint name="upper_trunk_to_neck" type="fixed">
         <origin rpy="0 0 0" xyz="0 0 ${l_upper_trunk}"/>
         <parent link="upper_trunk"/>
@@ -185,5 +185,5 @@
         </inertial> -->
     </link>
-    <joint name="joint_head" type="fixed">
+    <joint name="neck_to_head" type="fixed">
         <origin rpy="0 0 0" xyz="0 0 ${l_neck}"/>
         <parent link="neck"/>
@@ -213,4 +213,60 @@
         </inertial>
     </link>
+    <joint name="left_forearm_to_hand" type="fixed">
+        <origin rpy="0 0 0" xyz="0 0 ${-l_forearm}"/>
+        <parent link="left_forearm"/>
+        <child link="left_hand"/>
+    </joint>
+    <link name="left_hand">
+        <visual>
+        <origin rpy="0 ${pi/2} 0" xyz="${r_forearm/2} 0 ${-thickness/2}"/>
+        <geometry>
+            <box size="${l_hand} ${w_hand} ${thickness}"/>
+        </geometry>
+        <material name="white"/>
+        </visual>
+        <collision>
+        <origin rpy="0 ${pi/2} 0" xyz="0 0 ${-thickness/2}"/>
+        <geometry>
+            <box size="${l_hand} ${w_hand} ${thickness}"/>
+        </geometry>
+        </collision>
+        <inertial>
+        <origin rpy="0 ${pi/2} 0" xyz="0 0 ${-l_forearm/2}"/>
+        <mass value="${m_hand}"/>
+        <inertia
+            ixx="${m_hand*(pow(thickness,2) + pow(w_hand,2))/12}" ixy="0.0" ixz="0.0"
+            iyy="${m_hand*(pow(l_hand,2) + pow(thickness,2))/12}" iyz="0.0"
+            izz="${m_hand*(pow(l_hand,2) + pow(w_hand,2))/12}"/>
+        </inertial>
+    </link>
+    <joint name="right_forearm_to_hand" type="fixed">
+        <origin rpy="0 0 0" xyz="0 0 ${-l_forearm}"/>
+        <parent link="right_forearm"/>
+        <child link="right_hand"/>
+    </joint>
+    <link name="right_hand">
+        <visual>
+        <origin rpy="0 ${pi/2} 0" xyz="${r_forearm/2} 0 ${-thickness/2}"/>
+        <geometry>
+            <box size="${l_hand} ${w_hand} ${thickness}"/>
+        </geometry>
+        <material name="white"/>
+        </visual>
+        <collision>
+        <origin rpy="0 ${pi/2} 0" xyz="0 0 ${-thickness/2}"/>
+        <geometry>
+            <box size="${l_hand} ${w_hand} ${thickness}"/>
+        </geometry>
+        </collision>
+        <inertial>
+        <origin rpy="0 ${pi/2} 0" xyz="0 0 ${-l_forearm/2}"/>
+        <mass value="${m_hand}"/>
+        <inertia
+            ixx="${m_hand*(pow(thickness,2) + pow(w_hand,2))/12}" ixy="0.0" ixz="0.0"
+            iyy="${m_hand*(pow(l_hand,2) + pow(thickness,2))/12}" iyz="0.0"
+            izz="${m_hand*(pow(l_hand,2) + pow(w_hand,2))/12}"/>
+        </inertial>
+    </link>
 </xacro:macro>
 </robot>

File: urdf/macros/measurements.xacro (robot description, xacro)
@@ -16,5 +16,5 @@
   <xacro:property name="whole_body" value="1.7268" />
   <xacro:property name="thickness" value="0.02" />
-  <xacro:property name="r_neck" value="${l_neck/2}" />
+  <xacro:property name="r_neck" value="${l_neck/1.5}" />
   <xacro:property name="r_head" value="0.15" />
   <xacro:property name="r_upper_trunk" value="${l_upper_trunk/2}" />
@@ -22,5 +22,5 @@
   <xacro:property name="r_upper_arm" value="${l_upper_arm/6.5}" />
   <xacro:property name="r_forearm" value="${l_forearm/7}" />
-  <xacro:property name="w_hand" value="${l_hand/3}" />
+  <xacro:property name="w_hand" value="${l_hand/4}" />
   <xacro:property name="r_thigh" value="${l_thigh/4.5}" />
   <xacro:property name="r_shank" value="${l_shank/5.5}" />

Commit message: LEFT and RIGHT are mirrored

File: urdf/human/human_lower.xacro (robot description, xacro)
@@ -30,10 +30,10 @@
         </inertial>
     </link>
-    <joint name="lower_trunk_to_left_thigh" type="fixed">
+    <joint name="lower_trunk_to_right_thigh" type="fixed">
         <origin rpy="0 0 0" xyz="0 ${-r_lower_trunk/2} ${-l_lower_trunk/2}"/>
         <parent link="lower_trunk"/>
-        <child link="left_thigh"/>
-    </joint>
-    <link name="left_thigh">
+        <child link="right_thigh"/>
+    </joint>
+    <link name="right_thigh">
         <visual>
         <origin rpy="0 0 0" xyz="0 0 ${-l_thigh/2}"/>
@@ -58,10 +58,10 @@
         </inertial>
     </link>
-    <joint name="lower_trunk_to_right_thigh" type="fixed">
+    <joint name="lower_trunk_to_left_thigh" type="fixed">
         <origin rpy="0 0 0" xyz="0 ${r_lower_trunk/2} ${-l_lower_trunk/2}"/>
         <parent link="lower_trunk"/>
-        <child link="right_thigh"/>
-    </joint>
-    <link name="right_thigh">
+        <child link="left_thigh"/>
+    </joint>
+    <link name="left_thigh">
         <visual>
         <origin rpy="0 0 0" xyz="0 0 ${-l_thigh/2}"/>
@@ -86,5 +86,61 @@
         </inertial>
     </link>
-    <joint name="left_thight_to_shank" type="fixed">
+    <joint name="right_thight_to_shank" type="fixed">
+        <origin rpy="0 0 0" xyz="0 0 ${-l_thigh}"/>
+        <parent link="right_thigh"/>
+        <child link="right_shank"/>
+    </joint>
+    <link name="right_shank">
+        <visual>
+        <origin rpy="0 0 0" xyz="0 0 ${-l_shank/2}"/>
+        <geometry>
+            <cylinder length="${l_shank}" radius="${r_shank}"/>
+        </geometry>
+        <material name="white"/>
+        </visual>
+        <collision>
+        <origin rpy="0 0 0" xyz="0 0 ${-l_shank/2}"/>
+        <geometry>
+            <cylinder length="${l_shank}" radius="${r_shank}"/>
+        </geometry>
+        </collision>
+        <inertial>
+        <origin rpy="0 0 0" xyz="0 0 ${-l_shank/2}"/>
+        <mass value="${m_shank}"/>
+        <inertia
+            ixx="${m_shank*(3*pow(r_shank,2)+pow(l_shank,2))/12}" ixy="0.0" ixz="0.0"
+            iyy="${m_shank*(3*pow(r_shank,2)+pow(l_shank,2))/12}" iyz="0.0"
+            izz="${m_shank*pow(r_shank,2)/2}"/>
+        </inertial>
+    </link>
+    <joint name="right_shank_to_foot" type="fixed">
+        <origin rpy="0 0 0" xyz="0 0 ${-l_shank}"/>
+        <parent link="right_shank"/>
+        <child link="right_foot"/>
+    </joint>
+    <link name="right_foot">
+        <visual>
+        <origin rpy="0 0 0" xyz="${r_shank/2} 0 ${-thickness/2}"/>
+        <geometry>
+            <box size="${l_foot} ${w_foot} ${thickness}"/>
+        </geometry>
+        <material name="white"/>
+        </visual>
+        <collision>
+        <origin rpy="0 0 0" xyz="0 0 ${-thickness/2}"/>
+        <geometry>
+            <box size="${l_foot} ${w_foot} ${thickness}"/>
+        </geometry>
+        </collision>
+        <inertial>
+        <origin rpy="0 0 0" xyz="0 0 ${-l_shank/2}"/>
+        <mass value="${m_foot}"/>
+        <inertia
+            ixx="${m_foot*(pow(thickness,2) + pow(w_foot,2))/12}" ixy="0.0" ixz="0.0"
+            iyy="${m_foot*(pow(l_foot,2) + pow(thickness,2))/12}" iyz="0.0"
+            izz="${m_foot*(pow(l_foot,2) + pow(w_foot,2))/12}"/>
+        </inertial>
+    </link>
+        <joint name="left_thight_to_shank" type="fixed">
         <origin rpy="0 0 0" xyz="0 0 ${-l_thigh}"/>
         <parent link="left_thigh"/>
@@ -142,60 +198,4 @@
         </inertial>
     </link>
-        <joint name="right_thight_to_shank" type="fixed">
-        <origin rpy="0 0 0" xyz="0 0 ${-l_thigh}"/>
-        <parent link="right_thigh"/>
-        <child link="right_shank"/>
-    </joint>
-    <link name="right_shank">
-        <visual>
-        <origin rpy="0 0 0" xyz="0 0 ${-l_shank/2}"/>
-        <geometry>
-            <cylinder length="${l_shank}" radius="${r_shank}"/>
-        </geometry>
-        <material name="white"/>
-        </visual>
-        <collision>
-        <origin rpy="0 0 0" xyz="0 0 ${-l_shank/2}"/>
-        <geometry>
-            <cylinder length="${l_shank}" radius="${r_shank}"/>
-        </geometry>
-        </collision>
-        <inertial>
-        <origin rpy="0 0 0" xyz="0 0 ${-l_shank/2}"/>
-        <mass value="${m_shank}"/>
-        <inertia
-            ixx="${m_shank*(3*pow(r_shank,2)+pow(l_shank,2))/12}" ixy="0.0" ixz="0.0"
-            iyy="${m_shank*(3*pow(r_shank,2)+pow(l_shank,2))/12}" iyz="0.0"
-            izz="${m_shank*pow(r_shank,2)/2}"/>
-        </inertial>
-    </link>
-    <joint name="right_shank_to_foot" type="fixed">
-        <origin rpy="0 0 0" xyz="0 0 ${-l_shank}"/>
-        <parent link="right_shank"/>
-        <child link="right_foot"/>
-    </joint>
-    <link name="right_foot">
-        <visual>
-        <origin rpy="0 0 0" xyz="${r_shank/2} 0 ${-thickness/2}"/>
-        <geometry>
-            <box size="${l_foot} ${w_foot} ${thickness}"/>
-        </geometry>
-        <material name="white"/>
-        </visual>
-        <collision>
-        <origin rpy="0 0 0" xyz="0 0 ${-thickness/2}"/>
-        <geometry>
-            <box size="${l_foot} ${w_foot} ${thickness}"/>
-        </geometry>
-        </collision>
-        <inertial>
-        <origin rpy="0 0 0" xyz="0 0 ${-l_shank/2}"/>
-        <mass value="${m_foot}"/>
-        <inertia
-            ixx="${m_foot*(pow(thickness,2) + pow(w_foot,2))/12}" ixy="0.0" ixz="0.0"
-            iyy="${m_foot*(pow(l_foot,2) + pow(thickness,2))/12}" iyz="0.0"
-            izz="${m_foot*(pow(l_foot,2) + pow(w_foot,2))/12}"/>
-        </inertial>
-    </link>
 </xacro:macro>
 </robot>

File: urdf/human/human_upper.xacro (robot description, xacro)
@@ -28,8 +28,8 @@
         </inertial>
     </link>
-    <xacro:spherical name="left_shoulder" parent="upper_trunk" child="left_upper_arm" x="1" y="1" z="1">
+    <xacro:spherical name="right_shoulder" parent="upper_trunk" child="right_upper_arm" x="1" y="1" z="1">
         <origin rpy="0 0 0" xyz="0 ${-r_upper_trunk} ${l_upper_trunk}"/>
     </xacro:spherical>
-    <link name="left_upper_arm">
+    <link name="right_upper_arm">
         <visual>
         <origin rpy="0 0 0" xyz="0 0 ${-l_upper_arm/2}"/>
@@ -59,8 +59,8 @@
         </inertial> -->
     </link>
-    <xacro:spherical name="right_shoulder" parent="upper_trunk" child="right_upper_arm" x="-1" y="1" z="-1">
+    <xacro:spherical name="left_shoulder" parent="upper_trunk" child="left_upper_arm" x="-1" y="1" z="-1">
         <origin rpy="0 0 0" xyz="0 ${r_upper_trunk} ${l_upper_trunk}"/>
     </xacro:spherical>
-    <link name="right_upper_arm">
+    <link name="left_upper_arm">
         <visual>
         <origin rpy="0 0 0" xyz="0 0 ${-l_upper_arm/2}"/>
@@ -90,8 +90,8 @@
         </inertial> -->
     </link>
-    <xacro:spherical name="left_elbow" parent="left_upper_arm" child="left_forearm" x="fixed" y="1" z="1">
+    <xacro:spherical name="right_elbow" parent="right_upper_arm" child="right_forearm" x="fixed" y="1" z="1">
         <origin rpy="0 0 0" xyz="0 0 ${-l_upper_arm}"/>
     </xacro:spherical>
-    <link name="left_forearm">
+    <link name="right_forearm">
         <visual>
         <origin rpy="0 0 0" xyz="0 0 ${-l_forearm/2}"/>
@@ -121,8 +121,8 @@
         </inertial> -->
     </link>
-    <xacro:spherical name="right_elbow" parent="right_upper_arm" child="right_forearm" x="fixed" y="1" z="-1">
+    <xacro:spherical name="left_elbow" parent="left_upper_arm" child="left_forearm" x="fixed" y="1" z="-1">
         <origin rpy="0 0 0" xyz="0 0 ${-l_upper_arm}"/>
     </xacro:spherical>
-    <link name="right_forearm">
+    <link name="left_forearm">
         <visual>
         <origin rpy="0 0 0" xyz="0 0 ${-l_forearm/2}"/>
@@ -213,12 +213,40 @@
         </inertial>
     </link>
-    <!-- <joint name="left_forearm_to_hand" type="fixed">
+    <!-- <joint name="right_forearm_to_hand" type="fixed">
+        <origin rpy="0 0 0" xyz="0 0 ${-l_forearm}"/>
+        <parent link="right_forearm"/>
+        <child link="right_hand"/>
+    </joint> -->
+    <xacro:spherical name="right_wrist" parent="right_forearm" child="right_hand" x="1" y="1" z="1">
+        <origin rpy="0 0 0" xyz="0 0 ${-l_forearm}"/>
+    </xacro:spherical>
+    <link name="right_hand">
+        <visual>
+        <origin rpy="0 ${pi/2} 0" xyz="${r_forearm/2} 0 ${-thickness/2}"/>
+        <geometry>
+            <box size="${l_hand} ${w_hand} ${thickness}"/>
+        </geometry>
+        <material name="white"/>
+        </visual>
+        <collision>
+        <origin rpy="0 ${pi/2} 0" xyz="0 0 ${-thickness/2}"/>
+        <geometry>
+            <box size="${l_hand} ${w_hand} ${thickness}"/>
+        </geometry>
+        </collision>
+        <inertial>
+        <origin rpy="0 ${pi/2} 0" xyz="0 0 ${-l_forearm/2}"/>
+        <mass value="${m_hand}"/>
+        <inertia
+            ixx="${m_hand*(pow(thickness,2) + pow(w_hand,2))/12}" ixy="0.0" ixz="0.0"
+            iyy="${m_hand*(pow(l_hand,2) + pow(thickness,2))/12}" iyz="0.0"
+            izz="${m_hand*(pow(l_hand,2) + pow(w_hand,2))/12}"/>
+        </inertial>
+    </link>
+    <joint name="left_forearm_to_hand" type="fixed">
         <origin rpy="0 0 0" xyz="0 0 ${-l_forearm}"/>
         <parent link="left_forearm"/>
         <child link="left_hand"/>
-    </joint> -->
-    <xacro:spherical name="left_wrist" parent="left_forearm" child="left_hand" x="1" y="1" z="1">
-        <origin rpy="0 0 0" xyz="0 0 ${-l_forearm}"/>
-    </xacro:spherical>
+    </joint>
     <link name="left_hand">
         <visual>
@@ -244,32 +272,4 @@
         </inertial>
     </link>
-    <joint name="right_forearm_to_hand" type="fixed">
-        <origin rpy="0 0 0" xyz="0 0 ${-l_forearm}"/>
-        <parent link="right_forearm"/>
-        <child link="right_hand"/>
-    </joint>
-    <link name="right_hand">
-        <visual>
-        <origin rpy="0 ${pi/2} 0" xyz="${r_forearm/2} 0 ${-thickness/2}"/>
-        <geometry>
-            <box size="${l_hand} ${w_hand} ${thickness}"/>
-        </geometry>
-        <material name="white"/>
-        </visual>
-        <collision>
-        <origin rpy="0 ${pi/2} 0" xyz="0 0 ${-thickness/2}"/>
-        <geometry>
-            <box size="${l_hand} ${w_hand} ${thickness}"/>
-        </geometry>
-        </collision>
-        <inertial>
-        <origin rpy="0 ${pi/2} 0" xyz="0 0 ${-l_forearm/2}"/>
-        <mass value="${m_hand}"/>
-        <inertia
-            ixx="${m_hand*(pow(thickness,2) + pow(w_hand,2))/12}" ixy="0.0" ixz="0.0"
-            iyy="${m_hand*(pow(l_hand,2) + pow(thickness,2))/12}" iyz="0.0"
-            izz="${m_hand*(pow(l_hand,2) + pow(w_hand,2))/12}"/>
-        </inertial>
-    </link>
 </xacro:macro>
 </robot>
