Commit message: left upper arm added but lower trunk width should change

File: urdf/human/human_upper.xacro (robot description, xacro)
@@ -3,5 +3,5 @@
     <xacro:macro name="human_upper">
     <xacro:spherical name="base_to_upper_trunk" parent="base_link" child="upper_trunk">
-        <origin rpy="0.0 0.0 0.0" xyz="0 0 ${thickness+l_shank+l_thigh+l_lower_trunk}"/>
+        <origin rpy="0 0 0" xyz="0 0 ${thickness+l_shank+l_thigh+l_lower_trunk}"/>
     </xacro:spherical>
     <link name="upper_trunk">
@@ -28,40 +28,30 @@
         </inertial>
     </link>
+    <xacro:spherical name="left_shoulder" parent="upper_trunk" child="left_upper_arm">
+        <origin rpy="0 0 0" xyz="0 ${-r_upper_trunk} ${l_upper_trunk}"/>
+    </xacro:spherical>
+    <link name="left_upper_arm">
+        <visual>
+        <origin rpy="0 0 0" xyz="0 0 ${-l_upper_arm/2}"/>
+        <geometry>
+            <cylinder length="${l_upper_arm}" radius="${r_upper_arm}"/>
+        </geometry>
+        <material name="blue"/>
+        </visual>
+        <collision>
+        <origin rpy="0 0 0" xyz="0 0 ${-l_upper_arm/2}"/>
+        <geometry>
+            <cylinder length="${l_upper_arm}" radius="${r_upper_arm}"/>
+        </geometry>
+        </collision>
+        <inertial>
+        <origin rpy="0 0 0" xyz="0 0 ${-l_upper_arm/2}"/>
+        <mass value="${m_upper_arm}"/>
+        <inertia
+            ixx="${m_upper_arm*(3*pow(r_upper_arm,2)+pow(l_upper_arm,2))/12}" ixy="0.0" ixz="0.0"
+            iyy="${m_upper_arm*(3*pow(r_upper_arm,2)+pow(l_upper_arm,2))/12}" iyz="0.0"
+            izz="${m_upper_arm*pow(r_upper_arm,2)/2}"/>
+        </inertial>
+    </link>
 </xacro:macro>
 </robot>
-  <!-- <xacro:spherical name="base_to_lower_trunk" parent="base_link" child="lower_trunk">
-    <origin rpy="0.0 0.0 0.0" xyz="0 0 1"/>
-  </xacro:spherical> -->
-  <!-- <joint name="joint_1" type="revolute">
-    <origin xyz="0 0 ${radius}" rpy="0 0 0" />
-    <axis xyz="0 1 0"/>
-    <parent link="base_link"/>
-    <child link="link_01"/>
-    <limit effort="1" lower="-1.57079632679" upper="1.57079632679" velocity="1"/>
-  </joint> -->
-  <!--<xacro:cylindrical_part name="link_02" density="1" cm="1" length="5" radius="2">
-    <origin rpy="0 0 0" xyz="0 0 0"/>
-  </xacro:cylindrical_part>-->
-  <!-- <link name="link_01">
-      <visual>
-        <origin xyz="0 0 ${2*radius}" rpy="0 0 0" />
-        <geometry>
-          <cylinder length="${l_upper_arm}" radius="${w_upper_arm}"/>
-        </geometry>
-        <material name="blue" />
-      </visual>
-      <collision>
-        <origin xyz="0 0 ${2*radius}" rpy="0 0 0" />
-        <geometry>
-          <cylinder length="${l_upper_arm}" radius="${w_upper_arm}"/>
-        </geometry>
-      </collision>
-      <inertial>
-        <origin xyz="0 0 ${2*radius}" rpy="0 0 0" />
-        <mass value="${mass}"/>
-        <inertia
-          ixx="${mass*(3*pow(w_upper_arm,2)+pow(l_upper_arm,2))/12}" ixy="0.0" ixz="0.0"
-          iyy="${mass*(3*pow(w_upper_arm,2)+pow(l_upper_arm,2))/12}" iyz="0.0"
-          izz="${mass*pow(w_upper_arm,2)/2}"/>
-      </inertial>
-    </link> -->

File: urdf/macros/measurements.xacro (robot description, xacro)
@@ -17,6 +17,6 @@
   <xacro:property name="r_upper_trunk" value="${l_upper_trunk/2}" />
   <xacro:property name="r_lower_trunk" value="${l_lower_trunk*1.25}" />
-  <xacro:property name="r_upper_arm" value="${l_upper_arm/3}" />
-  <xacro:property name="r_forearm" value="${l_forearm/3}" />
+  <xacro:property name="r_upper_arm" value="${l_upper_arm/6}" />
+  <xacro:property name="r_forearm" value="${l_forearm/7}" />
   <xacro:property name="w_hand" value="${l_hand/3}" />
   <xacro:property name="r_thigh" value="${l_thigh/5}" />

Commit message: spherical macro, shoulder and trunk axes fixed

File: urdf/human/human_upper.xacro (robot description, xacro)
@@ -2,5 +2,5 @@
 <robot xmlns:xacro="http://www.ros.org/wiki/xacro">
     <xacro:macro name="human_upper">
-    <xacro:spherical name="base_to_upper_trunk" parent="base_link" child="upper_trunk">
+    <xacro:spherical name="base_to_upper_trunk" parent="base_link" child="upper_trunk" x="1" y="-1" z="1">
         <origin rpy="0 0 0" xyz="0 0 ${thickness+l_shank+l_thigh+l_lower_trunk}"/>
     </xacro:spherical>
@@ -28,5 +28,5 @@
         </inertial>
     </link>
-    <xacro:spherical name="left_shoulder" parent="upper_trunk" child="left_upper_arm">
+    <xacro:spherical name="left_shoulder" parent="upper_trunk" child="left_upper_arm" x="1" y="1" z="1">
         <origin rpy="0 0 0" xyz="0 ${-r_upper_trunk} ${l_upper_trunk}"/>
     </xacro:spherical>
@@ -54,4 +54,30 @@
         </inertial>
     </link>
+    <xacro:spherical name="right_shoulder" parent="upper_trunk" child="right_upper_arm" x="-1" y="1" z="-1">
+        <origin rpy="0 0 0" xyz="0 ${r_upper_trunk} ${l_upper_trunk}"/>
+    </xacro:spherical>
+    <link name="right_upper_arm">
+        <visual>
+        <origin rpy="0 0 0" xyz="0 0 ${-l_upper_arm/2}"/>
+        <geometry>
+            <cylinder length="${l_upper_arm}" radius="${r_upper_arm}"/>
+        </geometry>
+        <material name="blue"/>
+        </visual>
+        <collision>
+        <origin rpy="0 0 0" xyz="0 0 ${-l_upper_arm/2}"/>
+        <geometry>
+            <cylinder length="${l_upper_arm}" radius="${r_upper_arm}"/>
+        </geometry>
+        </collision>
+        <inertial>
+        <origin rpy="0 0 0" xyz="0 0 ${-l_upper_arm/2}"/>
+        <mass value="${m_upper_arm}"/>
+        <inertia
+            ixx="${m_upper_arm*(3*pow(r_upper_arm,2)+pow(l_upper_arm,2))/12}" ixy="0.0" ixz="0.0"
+            iyy="${m_upper_arm*(3*pow(r_upper_arm,2)+pow(l_upper_arm,2))/12}" iyz="0.0"
+            izz="${m_upper_arm*pow(r_upper_arm,2)/2}"/>
+        </inertial>
+    </link>
 </xacro:macro>
 </robot>

File: urdf/macros/spherical.xacro (robot description, xacro)
@@ -1,8 +1,8 @@
 <?xml version="1.0"?>
 <robot xmlns:xacro="http://www.ros.org/wiki/xacro">
-<xacro:macro name="spherical" params="name parent child *origin">
+<xacro:macro name="spherical" params="name parent child x y z *origin">
     <joint name="${name}_y" type="revolute">
       <xacro:insert_block name="origin" />
-      <axis xyz="0 1 0" />
+      <axis xyz="0 ${y} 0" />
       <limit effort="1000.0" lower="-3.14" upper="3.14" velocity="0.5"/>
       <parent link="${parent}"/>
@@ -16,5 +16,5 @@
     </link>
     <joint name="${name}_x" type="revolute">
-      <axis xyz="1 0 0" />
+      <axis xyz="${x} 0 0" />
       <limit effort="1000.0" lower="-3.14" upper="3.14" velocity="0.5"/>
       <parent link="${name}_virt_link_1"/>
@@ -28,5 +28,5 @@
     </link>
     <joint name="${name}_z" type="revolute">
-      <axis xyz="0 0 1" />
+      <axis xyz="0 0 ${z}" />
       <limit effort="1000.0" lower="-3.14" upper="3.14" velocity="0.5"/>
       <parent link="${name}_virt_link_2"/>

Commit message: left elbow 2 dof. Spherical macro updated with xacro:if

File: urdf/human/human_upper.xacro (robot description, xacro)
@@ -80,5 +80,5 @@
         </inertial>
     </link>
-    <xacro:spherical name="left_elbow" parent="left_upper_arm" child="left_forearm" x="0" y="1" z="-1">
+    <xacro:spherical name="left_elbow" parent="left_upper_arm" child="left_forearm" x="fixed" y="1" z="1">
         <origin rpy="0 0 0" xyz="0 0 ${-l_upper_arm}"/>
     </xacro:spherical>

File: urdf/macros/spherical.xacro (robot description, xacro)
@@ -15,10 +15,18 @@
       </inertial>
     </link>
-    <joint name="${name}_x" type="revolute">
-      <axis xyz="${x} 0 0" />
-      <limit effort="1000.0" lower="-3.14" upper="3.14" velocity="0.5"/>
-      <parent link="${name}_virt_link_1"/>
-      <child link="${name}_virt_link_2"/>
-    </joint>
+    <xacro:if value="${x == 'fixed'}">
+      <joint name="${name}_x" type="fixed">
+        <parent link="${name}_virt_link_1"/>
+        <child link="${name}_virt_link_2"/>
+      </joint>
+    </xacro:if>
+    <xacro:unless value="${x == 'fixed'}">
+      <joint name="${name}_x" type="revolute">
+        <axis xyz="${x} 0 0" />
+        <limit effort="1000.0" lower="-3.14" upper="3.14" velocity="0.5"/>
+        <parent link="${name}_virt_link_1"/>
+        <child link="${name}_virt_link_2"/>
+      </joint>
+    </xacro:unless>
     <link name="${name}_virt_link_2">
       <inertial>

Commit message: right elbow added

File: urdf/human/human_upper.xacro (robot description, xacro)
@@ -106,4 +106,30 @@
         </inertial>
     </link>
+    <xacro:spherical name="right_elbow" parent="right_upper_arm" child="right_forearm" x="fixed" y="1" z="-1">
+        <origin rpy="0 0 0" xyz="0 0 ${-l_upper_arm}"/>
+    </xacro:spherical>
+    <link name="right_forearm">
+        <visual>
+        <origin rpy="0 0 0" xyz="0 0 ${-l_forearm/2}"/>
+        <geometry>
+            <cylinder length="${l_forearm}" radius="${r_forearm}"/>
+        </geometry>
+        <material name="orange"/>
+        </visual>
+        <collision>
+        <origin rpy="0 0 0" xyz="0 0 ${-l_forearm/2}"/>
+        <geometry>
+            <cylinder length="${l_forearm}" radius="${r_forearm}"/>
+        </geometry>
+        </collision>
+        <inertial>
+        <origin rpy="0 0 0" xyz="0 0 ${-l_forearm/2}"/>
+        <mass value="${m_forearm}"/>
+        <inertia
+            ixx="${m_forearm*(3*pow(r_forearm,2)+pow(l_forearm,2))/12}" ixy="0.0" ixz="0.0"
+            iyy="${m_forearm*(3*pow(r_forearm,2)+pow(l_forearm,2))/12}" iyz="0.0"
+            izz="${m_forearm*pow(r_upper_arm,2)/2}"/>
+        </inertial>
+    </link>
 </xacro:macro>
 </robot>

Commit message: ok, the crash problem was due to PID. Now works but marginally stable

File: urdf/human/human_upper.xacro (robot description, xacro)
@@ -48,8 +48,13 @@
         <origin rpy="0 0 0" xyz="0 0 ${-l_upper_arm/2}"/>
         <mass value="${m_upper_arm}"/>
-        <inertia
+        <!-- <inertia
             ixx="${m_upper_arm*(3*pow(r_upper_arm,2)+pow(l_upper_arm,2))/12}" ixy="0.0" ixz="0.0"
             iyy="${m_upper_arm*(3*pow(r_upper_arm,2)+pow(l_upper_arm,2))/12}" iyz="0.0"
             izz="${m_upper_arm*pow(r_upper_arm,2)/2}"/>
+        </inertial> -->
+        <inertia
+            ixx="${2*m_upper_arm*pow(r_upper_arm,2)/5}" ixy="0.0" ixz="0.0"
+            iyy="${2*m_upper_arm*pow(r_upper_arm,2)/5}" iyz="0.0"
+            izz="${2*m_upper_arm*pow(r_upper_arm,2)/5}"/>
         </inertial>
     </link>
@@ -74,8 +79,13 @@
         <origin rpy="0 0 0" xyz="0 0 ${-l_upper_arm/2}"/>
         <mass value="${m_upper_arm}"/>
-        <inertia
+        <!-- <inertia
             ixx="${m_upper_arm*(3*pow(r_upper_arm,2)+pow(l_upper_arm,2))/12}" ixy="0.0" ixz="0.0"
             iyy="${m_upper_arm*(3*pow(r_upper_arm,2)+pow(l_upper_arm,2))/12}" iyz="0.0"
             izz="${m_upper_arm*pow(r_upper_arm,2)/2}"/>
+        </inertial> -->
+        <inertia
+            ixx="${2*m_upper_arm*pow(r_upper_arm,2)/5}" ixy="0.0" ixz="0.0"
+            iyy="${2*m_upper_arm*pow(r_upper_arm,2)/5}" iyz="0.0"
+            izz="${2*m_upper_arm*pow(r_upper_arm,2)/5}"/>
         </inertial>
     </link>
@@ -100,8 +110,13 @@
         <origin rpy="0 0 0" xyz="0 0 ${-l_forearm/2}"/>
         <mass value="${m_forearm}"/>
-        <inertia
+        <!-- <inertia
             ixx="${m_forearm*(3*pow(r_forearm,2)+pow(l_forearm,2))/12}" ixy="0.0" ixz="0.0"
             iyy="${m_forearm*(3*pow(r_forearm,2)+pow(l_forearm,2))/12}" iyz="0.0"
             izz="${m_forearm*pow(r_upper_arm,2)/2}"/>
+        </inertial> -->
+        <inertia
+            ixx="${2*m_forearm*pow(r_forearm,2)/5}" ixy="0.0" ixz="0.0"
+            iyy="${2*m_forearm*pow(r_forearm,2)/5}" iyz="0.0"
+            izz="${2*m_forearm*pow(r_forearm,2)/5}"/>
         </inertial>
     </link>
@@ -126,8 +141,13 @@
         <origin rpy="0 0 0" xyz="0 0 ${-l_forearm/2}"/>
         <mass value="${m_forearm}"/>
-        <inertia
+        <!-- <inertia
             ixx="${m_forearm*(3*pow(r_forearm,2)+pow(l_forearm,2))/12}" ixy="0.0" ixz="0.0"
             iyy="${m_forearm*(3*pow(r_forearm,2)+pow(l_forearm,2))/12}" iyz="0.0"
             izz="${m_forearm*pow(r_upper_arm,2)/2}"/>
+        </inertial> -->
+        <inertia
+            ixx="${2*m_forearm*pow(r_forearm,2)/5}" ixy="0.0" ixz="0.0"
+            iyy="${2*m_forearm*pow(r_forearm,2)/5}" iyz="0.0"
+            izz="${2*m_forearm*pow(r_forearm,2)/5}"/>
         </inertial>
     </link>

Commit message: going back to cylindrical inertia

File: urdf/human/human_upper.xacro (robot description, xacro)
@@ -48,14 +48,14 @@
         <origin rpy="0 0 0" xyz="0 0 ${-l_upper_arm/2}"/>
         <mass value="${m_upper_arm}"/>
-        <!-- <inertia
+        <inertia
             ixx="${m_upper_arm*(3*pow(r_upper_arm,2)+pow(l_upper_arm,2))/12}" ixy="0.0" ixz="0.0"
             iyy="${m_upper_arm*(3*pow(r_upper_arm,2)+pow(l_upper_arm,2))/12}" iyz="0.0"
             izz="${m_upper_arm*pow(r_upper_arm,2)/2}"/>
-        </inertial> -->
-        <inertia
+        </inertial>
+        <!-- <inertia
             ixx="${2*m_upper_arm*pow(r_upper_arm,2)/5}" ixy="0.0" ixz="0.0"
             iyy="${2*m_upper_arm*pow(r_upper_arm,2)/5}" iyz="0.0"
             izz="${2*m_upper_arm*pow(r_upper_arm,2)/5}"/>
-        </inertial>
+        </inertial> -->
     </link>
     <xacro:spherical name="right_shoulder" parent="upper_trunk" child="right_upper_arm" x="-1" y="1" z="-1">
@@ -79,14 +79,14 @@
         <origin rpy="0 0 0" xyz="0 0 ${-l_upper_arm/2}"/>
         <mass value="${m_upper_arm}"/>
-        <!-- <inertia
+        <inertia
             ixx="${m_upper_arm*(3*pow(r_upper_arm,2)+pow(l_upper_arm,2))/12}" ixy="0.0" ixz="0.0"
             iyy="${m_upper_arm*(3*pow(r_upper_arm,2)+pow(l_upper_arm,2))/12}" iyz="0.0"
             izz="${m_upper_arm*pow(r_upper_arm,2)/2}"/>
-        </inertial> -->
-        <inertia
+        </inertial>
+        <!-- <inertia
             ixx="${2*m_upper_arm*pow(r_upper_arm,2)/5}" ixy="0.0" ixz="0.0"
             iyy="${2*m_upper_arm*pow(r_upper_arm,2)/5}" iyz="0.0"
             izz="${2*m_upper_arm*pow(r_upper_arm,2)/5}"/>
-        </inertial>
+        </inertial> -->
     </link>
     <xacro:spherical name="left_elbow" parent="left_upper_arm" child="left_forearm" x="fixed" y="1" z="1">
@@ -110,14 +110,14 @@
         <origin rpy="0 0 0" xyz="0 0 ${-l_forearm/2}"/>
         <mass value="${m_forearm}"/>
-        <!-- <inertia
+        <inertia
             ixx="${m_forearm*(3*pow(r_forearm,2)+pow(l_forearm,2))/12}" ixy="0.0" ixz="0.0"
             iyy="${m_forearm*(3*pow(r_forearm,2)+pow(l_forearm,2))/12}" iyz="0.0"
             izz="${m_forearm*pow(r_upper_arm,2)/2}"/>
-        </inertial> -->
-        <inertia
+        </inertial>
+        <!-- <inertia
             ixx="${2*m_forearm*pow(r_forearm,2)/5}" ixy="0.0" ixz="0.0"
             iyy="${2*m_forearm*pow(r_forearm,2)/5}" iyz="0.0"
             izz="${2*m_forearm*pow(r_forearm,2)/5}"/>
-        </inertial>
+        </inertial> -->
     </link>
     <xacro:spherical name="right_elbow" parent="right_upper_arm" child="right_forearm" x="fixed" y="1" z="-1">
@@ -141,14 +141,14 @@
         <origin rpy="0 0 0" xyz="0 0 ${-l_forearm/2}"/>
         <mass value="${m_forearm}"/>
-        <!-- <inertia
+        <inertia
             ixx="${m_forearm*(3*pow(r_forearm,2)+pow(l_forearm,2))/12}" ixy="0.0" ixz="0.0"
             iyy="${m_forearm*(3*pow(r_forearm,2)+pow(l_forearm,2))/12}" iyz="0.0"
             izz="${m_forearm*pow(r_upper_arm,2)/2}"/>
-        </inertial> -->
-        <inertia
+        </inertial>
+        <!-- <inertia
             ixx="${2*m_forearm*pow(r_forearm,2)/5}" ixy="0.0" ixz="0.0"
             iyy="${2*m_forearm*pow(r_forearm,2)/5}" iyz="0.0"
             izz="${2*m_forearm*pow(r_forearm,2)/5}"/>
-        </inertial>
+        </inertial> -->
     </link>
 </xacro:macro>

Commit message: neck and head added

File: urdf/human/human_upper.xacro (robot description, xacro)
@@ -152,4 +152,65 @@
         </inertial> -->
     </link>
+    <joint name="joint_neck" type="fixed">
+        <origin rpy="0 0 0" xyz="0 0 ${l_upper_trunk}"/>
+        <parent link="upper_trunk"/>
+        <child link="neck"/>
+    </joint>
+    <link name="neck">
+        <visual>
+        <origin rpy="0 0 0" xyz="0 0 ${l_neck/2}"/>
+        <geometry>
+            <cylinder length="${l_neck}" radius="${r_neck}"/>
+        </geometry>
+        <material name="orange"/>
+        </visual>
+        <collision>
+        <origin rpy="0 0 0" xyz="0 0 ${l_neck/2}"/>
+        <geometry>
+            <cylinder length="${l_neck}" radius="${r_neck}"/>
+        </geometry>
+        </collision>
+        <inertial>
+        <origin rpy="0 0 0" xyz="0 0 ${l_neck/2}"/>
+        <mass value="${m_neck}"/>
+        <inertia
+            ixx="${m_neck*(3*pow(r_neck,2)+pow(l_neck,2))/12}" ixy="0.0" ixz="0.0"
+            iyy="${m_neck*(3*pow(r_neck,2)+pow(l_neck,2))/12}" iyz="0.0"
+            izz="${m_neck*pow(r_upper_arm,2)/2}"/>
+        </inertial>
+        <!-- <inertia
+            ixx="${2*m_neck*pow(r_neck,2)/5}" ixy="0.0" ixz="0.0"
+            iyy="${2*m_neck*pow(r_neck,2)/5}" iyz="0.0"
+            izz="${2*m_neck*pow(r_neck,2)/5}"/>
+        </inertial> -->
+    </link>
+    <joint name="joint_head" type="fixed">
+        <origin rpy="0 0 0" xyz="0 0 ${l_neck}"/>
+        <parent link="neck"/>
+        <child link="head"/>
+    </joint>
+    <link name="head">
+        <visual>
+        <origin rpy="0 0 0" xyz="0 0 ${r_head}"/>
+        <geometry>
+            <sphere radius="${r_head}"/>
+        </geometry>
+        <material name="blue"/>
+        </visual>
+        <collision>
+        <origin rpy="0 0 0" xyz="0 0 ${r_head}"/>
+        <geometry>
+            <sphere radius="${r_head}"/>
+        </geometry>
+        </collision>
+        <inertial>
+        <origin rpy="0 0 0" xyz="0 0 ${r_head}"/>
+        <mass value="${m_head}"/>
+        <inertia
+            ixx="${2*m_head*pow(r_head,2)/5}" ixy="0.0" ixz="0.0"
+            iyy="${2*m_head*pow(r_head,2)/5}" iyz="0.0"
+            izz="${2*m_head*pow(r_head,2)/5}"/>
+        </inertial>
+    </link>
 </xacro:macro>
 </robot>

File: urdf/macros/measurements.xacro (robot description, xacro)
@@ -2,5 +2,5 @@
 <robot name="human" xmlns:xacro="http://www.ros.org/wiki/xacro">
   <xacro:property name="l_neck" value="0.053" />
-  <xacro:property name="head" value="0.212-${neck}" />
+  <xacro:property name="head" value="0.212-${l_neck}" />
   <!-- <xacro:property name="l_upper_trunk" value="0.410" /> -->
   <xacro:property name="l_upper_trunk" value="0.510" />
@@ -17,5 +17,5 @@
   <xacro:property name="thickness" value="0.02" />
   <xacro:property name="r_neck" value="${l_neck/5}" />
-  <xacro:property name="r_head" value="${head/2}" />
+  <xacro:property name="r_head" value="0.15" />
   <xacro:property name="r_upper_trunk" value="${l_upper_trunk/1.5}" />
   <xacro:property name="r_lower_trunk" value="${l_lower_trunk*1.25}" />

Commit message: left wrist DOF added

File: urdf/human/human_upper.xacro (robot description, xacro)
@@ -213,9 +213,12 @@
         </inertial>
     </link>
-    <joint name="left_forearm_to_hand" type="fixed">
+    <!-- <joint name="left_forearm_to_hand" type="fixed">
         <origin rpy="0 0 0" xyz="0 0 ${-l_forearm}"/>
         <parent link="left_forearm"/>
         <child link="left_hand"/>
-    </joint>
+    </joint> -->
+    <xacro:spherical name="left_wrist" parent="left_forearm" child="left_hand" x="1" y="1" z="1">
+        <origin rpy="0 0 0" xyz="0 0 ${-l_forearm}"/>
+    </xacro:spherical>
     <link name="left_hand">
         <visual>

Commit message: both shoulders (corrected right hand :D ) work fine

File: urdf/human/human_upper.xacro (robot description, xacro)
@@ -213,12 +213,9 @@
         </inertial>
     </link>
-    <!-- <joint name="right_forearm_to_hand" type="fixed">
+    <joint name="right_forearm_to_hand" type="fixed">
         <origin rpy="0 0 0" xyz="0 0 ${-l_forearm}"/>
         <parent link="right_forearm"/>
         <child link="right_hand"/>
-    </joint> -->
-    <xacro:spherical name="right_wrist" parent="right_forearm" child="right_hand" x="1" y="1" z="1">
-        <origin rpy="0 0 0" xyz="0 0 ${-l_forearm}"/>
-    </xacro:spherical>
+    </joint>
     <link name="right_hand">
         <visual>
@@ -244,9 +241,12 @@
         </inertial>
     </link>
-    <joint name="left_forearm_to_hand" type="fixed">
+    <!-- <joint name="left_forearm_to_hand" type="fixed">
         <origin rpy="0 0 0" xyz="0 0 ${-l_forearm}"/>
         <parent link="left_forearm"/>
         <child link="left_hand"/>
-    </joint>
+    </joint> -->
+    <xacro:spherical name="left_wrist" parent="left_forearm" child="left_hand" x="1" y="1" z="1">
+        <origin rpy="0 0 0" xyz="0 0 ${-l_forearm}"/>
+    </xacro:spherical>
     <link name="left_hand">
         <visual>
