Commit message: spherical joint orders changed

File: urdf/macros/spherical.xacro (robot description, xacro)
@@ -2,7 +2,7 @@
 <robot xmlns:xacro="http://www.ros.org/wiki/xacro">
 <xacro:macro name="spherical" params="name parent child *origin">
-    <joint name="${name}_x" type="revolute">
+    <joint name="${name}_y" type="revolute">
       <xacro:insert_block name="origin" />
-      <axis xyz="1 0 0" />
+      <axis xyz="0 1 0" />
       <limit effort="1000.0" lower="-3.14" upper="3.14" velocity="0.5"/>
       <parent link="${parent}"/>
@@ -15,6 +15,6 @@
       </inertial>
     </link>
-    <joint name="${name}_y" type="revolute">
-      <axis xyz="0 1 0" />
+    <joint name="${name}_x" type="revolute">
+      <axis xyz="1 0 0" />
       <limit effort="1000.0" lower="-3.14" upper="3.14" velocity="0.5"/>
       <parent link="${name}_virt_link_1"/>
