Commit message: spherical virtual links naming (order might need to change)

File: urdf/macros/human.transmission.xacro (robot description, xacro)
@@ -3,5 +3,5 @@
   <transmission name="joint_1_1_tran1">
     <type>transmission_interface/SimpleTransmission</type>
-    <joint name="joint_1_1">
+    <joint name="joint_1_x">
       <hardwareInterface>hardware_interface/PositionJointInterface</hardwareInterface>
     </joint>
@@ -12,5 +12,5 @@
   <transmission name="joint_1_2_tran1">
     <type>transmission_interface/SimpleTransmission</type>
-    <joint name="joint_1_2">
+    <joint name="joint_1_y">
       <hardwareInterface>hardware_interface/PositionJointInterface</hardwareInterface>
     </joint>
@@ -21,5 +21,5 @@
   <transmission name="joint_1_3_tran1">
     <type>transmission_interface/SimpleTransmission</type>
-    <joint name="joint_1_3">
+    <joint name="joint_1_z">
       <hardwareInterface>hardware_interface/PositionJointInterface</hardwareInterface>
     </joint>

File: urdf/macros/spherical.xacro (robot description, xacro)
@@ -2,11 +2,11 @@
 <robot xmlns:xacro="http://www.ros.org/wiki/xacro">
 <xacro:macro name="spherical" params="name parent child *origin">
-    <joint name="${name}_1" type="revolute">
-      <axis xyz="-1 0 0" />
+    <joint name="${name}_x" type="revolute">
+      <axis xyz="1 0 0" />
       <limit effort="1000.0" lower="-3.14" upper="3.14" velocity="0.5"/>
       <parent link="${parent}"/>
-      <child link="${name}_virt_link_z"/>
+      <child link="${name}_virt_link_1"/>
     </joint>
-    <link name="${name}_virt_link_z">
+    <link name="${name}_virt_link_1">
       <inertial>
         <mass value="0.025" />
@@ -14,11 +14,11 @@
       </inertial>
     </link>
-    <joint name="${name}_2" type="revolute">
+    <joint name="${name}_y" type="revolute">
       <axis xyz="0 1 0" />
       <limit effort="1000.0" lower="-3.14" upper="3.14" velocity="0.5"/>
-      <parent link="${name}_virt_link_z"/>
-      <child link="${name}_virt_link_x"/>
+      <parent link="${name}_virt_link_1"/>
+      <child link="${name}_virt_link_2"/>
     </joint>
-    <link name="${name}_virt_link_x">
+    <link name="${name}_virt_link_2">
       <inertial>
         <mass value="0.025" />
@@ -26,11 +26,11 @@
       </inertial>
     </link>
-    <joint name="${name}_3" type="revolute">
+    <joint name="${name}_z" type="revolute">
       <axis xyz="0 0 1" />
       <limit effort="1000.0" lower="-3.14" upper="3.14" velocity="0.5"/>
-      <parent link="${name}_virt_link_x"/>
-      <child link="${name}_virt_link_y"/>
+      <parent link="${name}_virt_link_2"/>
+      <child link="${name}_virt_link_3"/>
     </joint>
-    <link name="${name}_virt_link_y">
+    <link name="${name}_virt_link_3">
       <inertial>
         <mass value="0.025" />
@@ -40,5 +40,5 @@
     <joint name="${name}_F" type="fixed">
       <xacro:insert_block name="origin" />
-      <parent link="${name}_virt_link_y"/>
+      <parent link="${name}_virt_link_3"/>
       <child link="${child}"/>
     </joint>

Commit message: controllers are also loaded succesfully

File: urdf/macros/human.transmission.xacro (robot description, xacro)
@@ -1,4 +1,85 @@
 <?xml version="1.0"?>
 <robot name="human" xmlns:xacro="http://www.ros.org/wiki/xacro">
+  <transmission name="base_to_upper_trunk_y_trans">
+    <type>transmission_interface/SimpleTransmission</type>
+    <joint name="base_to_upper_trunk_y">
+      <hardwareInterface>hardware_interface/PositionJointInterface</hardwareInterface>
+    </joint>
+    <actuator name="base_to_upper_trunk_y_motor">
+      <mechanicalReduction>1</mechanicalReduction>
+    </actuator>
+  </transmission>
+  <transmission name="base_to_upper_trunk_x_trans">
+    <type>transmission_interface/SimpleTransmission</type>
+    <joint name="base_to_upper_trunk_x">
+      <hardwareInterface>hardware_interface/PositionJointInterface</hardwareInterface>
+    </joint>
+    <actuator name="base_to_upper_trunk_x_motor">
+      <mechanicalReduction>1</mechanicalReduction>
+    </actuator>
+  </transmission>
+  <transmission name="base_to_upper_trunk_z_trans">
+    <type>transmission_interface/SimpleTransmission</type>
+    <joint name="base_to_upper_trunk_z">
+      <hardwareInterface>hardware_interface/PositionJointInterface</hardwareInterface>
+    </joint>
+    <actuator name="base_to_upper_trunk_z_motor">
+      <mechanicalReduction>1</mechanicalReduction>
+    </actuator>
+  </transmission>
+  <transmission name="left_shoulder_y_trans">
+    <type>transmission_interface/SimpleTransmission</type>
+    <joint name="left_shoulder_y">
+      <hardwareInterface>hardware_interface/PositionJointInterface</hardwareInterface>
+    </joint>
+    <actuator name="left_shoulder_y_motor">
+      <mechanicalReduction>1</mechanicalReduction>
+    </actuator>
+  </transmission>
+  <transmission name="left_shoulder_x_trans">
+    <type>transmission_interface/SimpleTransmission</type>
+    <joint name="left_shoulder_x">
+      <hardwareInterface>hardware_interface/PositionJointInterface</hardwareInterface>
+    </joint>
+    <actuator name="left_shoulder_x_motor">
+      <mechanicalReduction>1</mechanicalReduction>
+    </actuator>
+  </transmission>
+  <transmission name="left_shoulder_z_trans">
+    <type>transmission_interface/SimpleTransmission</type>
+    <joint name="left_shoulder_z">
+      <hardwareInterface>hardware_interface/PositionJointInterface</hardwareInterface>
+    </joint>
+    <actuator name="left_shoulder_z_motor">
+      <mechanicalReduction>1</mechanicalReduction>
+    </actuator>
+  </transmission>
+  <transmission name="right_shoulder_y_trans">
+    <type>transmission_interface/SimpleTransmission</type>
+    <joint name="right_shoulder_y">
+      <hardwareInterface>hardware_interface/PositionJointInterface</hardwareInterface>
+    </joint>
+    <actuator name="right_shoulder_y_motor">
+      <mechanicalReduction>1</mechanicalReduction>
+    </actuator>
+  </transmission>
+  <transmission name="right_shoulder_x_trans">
+    <type>transmission_interface/SimpleTransmission</type>
+    <joint name="right_shoulder_x">
+      <hardwareInterface>hardware_interface/PositionJointInterface</hardwareInterface>
+    </joint>
+    <actuator name="right_shoulder_x_motor">
+      <mechanicalReduction>1</mechanicalReduction>
+    </actuator>
+  </transmission>
+  <transmission name="right_shoulder_z_trans">
+    <type>transmission_interface/SimpleTransmission</type>
+    <joint name="right_shoulder_z">
+      <hardwareInterface>hardware_interface/PositionJointInterface</hardwareInterface>
+    </joint>
+    <actuator name="right_shoulder_z_motor">
+      <mechanicalReduction>1</mechanicalReduction>
+    </actuator>
+  </transmission>
   <!-- <transmission name="joint_1_1_tran1">
     <type>transmission_interface/SimpleTransmission</type>

Commit message: elbow controllers added but upper truck has fallen down

File: urdf/macros/human.transmission.xacro (robot description, xacro)
@@ -82,5 +82,5 @@
     </actuator>
   </transmission>
-  <!-- <transmission name="left_elbow_y_trans">
+  <transmission name="left_elbow_y_trans">
     <type>transmission_interface/SimpleTransmission</type>
     <joint name="left_elbow_y">
@@ -88,13 +88,4 @@
     </joint>
     <actuator name="left_elbow_y_motor">
-      <mechanicalReduction>1</mechanicalReduction>
-    </actuator>
-  </transmission>
-  <transmission name="left_elbow_x_trans">
-    <type>transmission_interface/SimpleTransmission</type>
-    <joint name="left_elbow_x">
-      <hardwareInterface>hardware_interface/PositionJointInterface</hardwareInterface>
-    </joint>
-    <actuator name="left_elbow_x_motor">
       <mechanicalReduction>1</mechanicalReduction>
     </actuator>
@@ -108,4 +99,22 @@
       <mechanicalReduction>1</mechanicalReduction>
     </actuator>
-  </transmission> -->
+  </transmission>
+  <transmission name="right_elbow_y_trans">
+    <type>transmission_interface/SimpleTransmission</type>
+    <joint name="right_elbow_y">
+      <hardwareInterface>hardware_interface/PositionJointInterface</hardwareInterface>
+    </joint>
+    <actuator name="right_elbow_y_motor">
+      <mechanicalReduction>1</mechanicalReduction>
+    </actuator>
+  </transmission>
+  <transmission name="right_elbow_z_trans">
+    <type>transmission_interface/SimpleTransmission</type>
+    <joint name="right_elbow_z">
+      <hardwareInterface>hardware_interface/PositionJointInterface</hardwareInterface>
+    </joint>
+    <actuator name="right_elbow_z_motor">
+      <mechanicalReduction>1</mechanicalReduction>
+    </actuator>
+  </transmission>
 </robot>
