Commit message: comparative rrbot additions

File: urdf/macros/human.gazebo.xacro (robot description, xacro)
@@ -1,8 +1,8 @@
 <?xml version="1.0"?>
-<robot xmlns:xacro="http://www.ros.org/wiki/xacro">
-  <xacro:macro name="human_gazebo">
+<robot name="human" xmlns:xacro="http://www.ros.org/wiki/xacro">
+  <xacro:macro name="human">
     <gazebo>
       <plugin name="gazebo_ros_control" filename="libgazebo_ros_control.so">
-        <robotNamespace>/human</robotNamespace>
+        <robotNamespace>human</robotNamespace>
       </plugin>
     </gazebo>

File: urdf/macros/human.transmission.xacro (robot description, xacro)
@@ -1,5 +1,5 @@
 <?xml version="1.0"?>
-<robot xmlns:xacro="http://www.ros.org/wiki/xacro">
-  <xacro:macro name="human_trans">
+<robot name="human" xmlns:xacro="http://www.ros.org/wiki/xacro">
+  <xacro:macro name="human">
     <transmission name="tran_1_1">
       <type>transmission_interface/SimpleTransmission</type>

File: urdf/macros/materials.xacro (robot description, xacro)
@@ -1,4 +1,4 @@
 <?xml version="1.0"?>
-<robot xmlns:xacro="http://www.ros.org/wiki/xacro">
+<robot name="human" xmlns:xacro="http://www.ros.org/wiki/xacro">
   <material name="blue">
     <color rgba="0 0 0.8 1"/>

File: urdf/macros/measurements.xacro (robot description, xacro)
@@ -1,4 +1,4 @@
 <?xml version="1.0"?>
-<robot xmlns:xacro="http://www.ros.org/wiki/xacro">
+<robot name="human" xmlns:xacro="http://www.ros.org/wiki/xacro">
   <xacro:property name="l_neck" value="0.053" />
   <xacro:property name="head" value="0.212-${neck}" />

Commit message: gazebo colors for now

File: urdf/macros/human.gazebo.xacro (robot description, xacro)
@@ -14,3 +14,51 @@
         <turnGravityOff>true</turnGravityOff>
     </gazebo>
+    <gazebo reference="head">
+       <material>Gazebo/Orange</material>
+    </gazebo>
+    <gazebo reference="neck">
+       <material>Gazebo/DarkOrangeTransparentOverlay</material>
+    </gazebo>
+    <gazebo reference="left_hand">
+       <material>Gazebo/Orange</material>
+    </gazebo>
+    <gazebo reference="right_hand">
+       <material>Gazebo/Orange</material>
+    </gazebo>
+    <gazebo reference="left_foot">
+       <material>Gazebo/Orange</material>
+    </gazebo>
+    <gazebo reference="right_foot">
+       <material>Gazebo/Orange</material>
+    </gazebo>
+    <gazebo reference="upper_trunk">
+       <material>Gazebo/Grass</material>
+    </gazebo>
+    <gazebo reference="lower_trunk">
+       <material>Gazebo/Green</material>
+    </gazebo>
+    <gazebo reference="left_thigh">
+       <material>Gazebo/Blue</material>
+    </gazebo>
+    <gazebo reference="right_thigh">
+       <material>Gazebo/Blue</material>
+    </gazebo>
+    <gazebo reference="left_shank">
+       <material>Gazebo/SkyBlue</material>
+    </gazebo>
+    <gazebo reference="right_shank">
+       <material>Gazebo/SkyBlue</material>
+    </gazebo>
+    <gazebo reference="left_upper_arm">
+       <material>Gazebo/Blue</material>
+    </gazebo>
+    <gazebo reference="left_forearm">
+       <material>Gazebo/SkyBlue</material>
+    </gazebo>
+    <gazebo reference="right_upper_arm">
+       <material>Gazebo/Blue</material>
+    </gazebo>
+    <gazebo reference="right_forearm">
+       <material>Gazebo/SkyBlue</material>
+    </gazebo>
 </robot>
