Commit message: unit_scale for kg to gr. Also to *0.1 to make gazebo stable. See descrip
https://answers.ros.org/question/216092/problem-with-the-robot-model-collapsing/

File: urdf/macros/measurements.xacro (robot description, xacro)
@@ -49,13 +49,14 @@
   <xacro:property name="m_base_link" value="0.01" />
   <xacro:property name="r_base_link" value="0.01" />
-  <xacro:property name="m_neck" value="${pi*l_neck*pow(r_neck,2)*d_neck*0.001}" />
-  <xacro:property name="m_head" value="${(4/3)*pi*pow(r_head,3)*0.001}" />
-  <xacro:property name="m_upper_trunk" value="${pi*l_upper_trunk*pow(r_upper_trunk,2)*d_upper_trunk*0.001}" />
-  <xacro:property name="m_lower_trunk" value="${pi*l_lower_trunk*pow(r_lower_trunk,2)*d_lower_trunk*0.001}" />
-  <xacro:property name="m_upper_arm" value="${pi*l_upper_arm*pow(r_upper_arm,2)*d_upper_arm*0.001}" />
-  <xacro:property name="m_forearm" value="${pi*l_forearm*pow(r_forearm,2)*d_forearm*0.001}" />
-  <xacro:property name="m_thigh" value="${pi*l_thigh*pow(r_thigh,2)*d_thigh*0.001}" />
-  <xacro:property name="m_shank" value="${pi*l_shank*pow(r_shank,2)*d_shank*0.001}" />
-  <xacro:property name="m_hand" value="${l_hand*w_hand*thickness*d_hand*0.001}" />
-  <xacro:property name="m_foot" value="${l_foot*w_foot*thickness*d_foot*0.001}" />
+  <xacro:property name="unit_scale" value="0.0001" />
+  <xacro:property name="m_neck" value="${pi*l_neck*pow(r_neck,2)*d_neck*unit_scale}" />
+  <xacro:property name="m_head" value="${(4/3)*pi*pow(r_head,3)*unit_scale}" />
+  <xacro:property name="m_upper_trunk" value="${pi*l_upper_trunk*pow(r_upper_trunk,2)*d_upper_trunk*unit_scale}" />
+  <xacro:property name="m_lower_trunk" value="${pi*l_lower_trunk*pow(r_lower_trunk,2)*d_lower_trunk*unit_scale}" />
+  <xacro:property name="m_upper_arm" value="${pi*l_upper_arm*pow(r_upper_arm,2)*d_upper_arm*unit_scale}" />
+  <xacro:property name="m_forearm" value="${pi*l_forearm*pow(r_forearm,2)*d_forearm*unit_scale}" />
+  <xacro:property name="m_thigh" value="${pi*l_thigh*pow(r_thigh,2)*d_thigh*unit_scale}" />
+  <xacro:property name="m_shank" value="${pi*l_shank*pow(r_shank,2)*d_shank*unit_scale}" />
+  <xacro:property name="m_hand" value="${l_hand*w_hand*thickness*d_hand*unit_scale}" />
+  <xacro:property name="m_foot" value="${l_foot*w_foot*thickness*d_foot*unit_scale}" />
 </robot>

Commit message: measurements update. Model is ready

File: urdf/macros/measurements.xacro (robot description, xacro)
@@ -16,13 +16,13 @@
   <xacro:property name="whole_body" value="1.7268" />
   <xacro:property name="thickness" value="0.02" />
-  <xacro:property name="r_neck" value="${l_neck/5}" />
+  <xacro:property name="r_neck" value="${l_neck/2}" />
   <xacro:property name="r_head" value="0.15" />
-  <xacro:property name="r_upper_trunk" value="${l_upper_trunk/1.5}" />
-  <xacro:property name="r_lower_trunk" value="${l_lower_trunk*1.25}" />
-  <xacro:property name="r_upper_arm" value="${l_upper_arm/6}" />
+  <xacro:property name="r_upper_trunk" value="${l_upper_trunk/2}" />
+  <xacro:property name="r_lower_trunk" value="${l_lower_trunk}" />
+  <xacro:property name="r_upper_arm" value="${l_upper_arm/6.5}" />
   <xacro:property name="r_forearm" value="${l_forearm/7}" />
   <xacro:property name="w_hand" value="${l_hand/3}" />
-  <xacro:property name="r_thigh" value="${l_thigh/4}" />
-  <xacro:property name="r_shank" value="${l_shank/5}" />
+  <xacro:property name="r_thigh" value="${l_thigh/4.5}" />
+  <xacro:property name="r_shank" value="${l_shank/5.5}" />
   <xacro:property name="w_foot" value="0.06" />
   <xacro:property name="cm_head" value="0.361" />

Commit message: yaml created, parameters are taken from it. launch+xacro updated

File: urdf/macros/measurements.xacro (robot description, xacro)
@@ -1,14 +1,15 @@
 <?xml version="1.0"?>
 <robot name="human" xmlns:xacro="http://www.ros.org/wiki/xacro">
+  <xacro:property name="human_params" value="${load_yaml('$(find imu_human_pkg)/config/human.yaml')}"/>
   <xacro:property name="l_neck" value="0.053" />
   <xacro:property name="head" value="0.212-${l_neck}" />
   <!-- <xacro:property name="l_upper_trunk" value="0.410" /> -->
-  <xacro:property name="l_upper_trunk" value="0.510" />
+  <xacro:property name="l_upper_trunk" value="${human_params['l_upper_trunk']}" />
   <!-- <xacro:property name="l_lower_trunk" value="0.135" /> -->
   <xacro:property name="l_lower_trunk" value="0.235" />
   <!-- <xacro:property name="l_upper_arm" value="0.65" /> -->
-  <xacro:property name="l_upper_arm" value="0.5" />
-  <xacro:property name="l_forearm" value="0.299" />
-  <xacro:property name="l_hand" value="0.203" />
+  <xacro:property name="l_upper_arm" value="${human_params['l_upper_arm']}" />
+  <xacro:property name="l_forearm" value="${human_params['l_forearm']}" />
+  <xacro:property name="l_hand" value="${human_params['l_hand']}" />
   <xacro:property name="l_thigh" value="0.449" />
   <xacro:property name="l_shank" value="0.429" />
