Commit message: REFACTORING! ur5e_gizem_moveit_config is under additionals

File: imu_human_pkg/urdf/human/human_upper.xacro (robot description, xacro)
@@ -220,5 +220,5 @@
     <link name="right_hand">
         <visual>
-        <origin rpy="0 ${pi/2} 0" xyz="${r_forearm/2} 0 ${-thickness/2}"/>
+        <origin rpy="${-pi/2} ${pi/2} 0" xyz="0 0 ${-l_hand/2}"/>
         <geometry>
             <box size="${l_hand} ${w_hand} ${thickness}"/>
@@ -227,11 +227,11 @@
         </visual>
         <collision>
-        <origin rpy="0 ${pi/2} 0" xyz="0 0 ${-thickness/2}"/>
-        <geometry>
-            <box size="${l_hand} ${w_hand} ${thickness}"/>
-        </geometry>
-        </collision>
-        <inertial>
-        <origin rpy="0 ${pi/2} 0" xyz="0 0 ${-l_forearm/2}"/>
+        <origin rpy="${-pi/2} ${pi/2} 0" xyz="0 0 ${-l_hand/2}"/>
+        <geometry>
+            <box size="${l_hand} ${w_hand} ${thickness}"/>
+        </geometry>
+        </collision>
+        <inertial>
+        <origin rpy="${-pi/2} ${pi/2} 0" xyz="0 0 ${-l_hand/2}"/>
         <mass value="${m_hand}"/>
         <inertia
@@ -251,5 +251,5 @@
     <link name="left_hand">
         <visual>
-        <origin rpy="0 ${pi/2} 0" xyz="${r_forearm/2} 0 ${-thickness/2}"/>
+        <origin rpy="${pi/2} ${pi/2} 0" xyz="0 0 ${-l_hand/2}"/>
         <geometry>
             <box size="${l_hand} ${w_hand} ${thickness}"/>
@@ -258,11 +258,11 @@
         </visual>
         <collision>
-        <origin rpy="0 ${pi/2} 0" xyz="0 0 ${-thickness/2}"/>
-        <geometry>
-            <box size="${l_hand} ${w_hand} ${thickness}"/>
-        </geometry>
-        </collision>
-        <inertial>
-        <origin rpy="0 ${pi/2} 0" xyz="0 0 ${-l_forearm/2}"/>
+        <origin rpy="${pi/2} ${pi/2} 0" xyz="0 0 ${-l_hand/2}"/>
+        <geometry>
+            <box size="${l_hand} ${w_hand} ${thickness}"/>
+        </geometry>
+        </collision>
+        <inertial>
+        <origin rpy="${pi/2} ${pi/2} 0" xyz="0 0 ${-l_hand/2}"/>
         <mass value="${m_hand}"/>
         <inertia
