Commit message: whoops human base link renamed

File: imu_human_pkg/urdf/human/human.urdf.xacro (robot description, xacro)
@@ -14,8 +14,8 @@
     <origin xyz="0 0 0" rpy="0 0 0" />
     <parent link="world"/>
-    <child link="base_link"/>
+    <child link="human_base_link"/>
     <origin rpy="0 0 0" xyz="0 0 0"/>
   </joint>
-  <link name="base_link">
+  <link name="human_base_link">
     <visual>
     <origin rpy="0 0 0" xyz="0 0 ${thickness+l_shank+l_thigh+l_lower_trunk/2}"/>

File: imu_human_pkg/urdf/human/human_lower.xacro (robot description, xacro)
@@ -4,5 +4,5 @@
     <joint name="base_to_lower_trunk" type="fixed">
         <origin rpy="0 0 0" xyz="0 0 ${thickness+l_shank+l_thigh+l_lower_trunk/2}"/>
-        <parent link="base_link"/>
+        <parent link="human_base_link"/>
         <child link="lower_trunk"/>
     </joint>

File: imu_human_pkg/urdf/human/human_upper.xacro (robot description, xacro)
@@ -2,5 +2,5 @@
 <robot xmlns:xacro="http://www.ros.org/wiki/xacro">
     <xacro:macro name="human_upper">
-    <xacro:spherical name="base_to_upper_trunk" parent="base_link" child="upper_trunk" x="1" y="-1" z="1">
+    <xacro:spherical name="base_to_upper_trunk" parent="human_base_link" child="upper_trunk" x="1" y="-1" z="1">
         <origin rpy="0 0 0" xyz="0 0 ${thickness+l_shank+l_thigh+l_lower_trunk}"/>
     </xacro:spherical>
