Commit message: follow_joint_trajectory WORKS!!

File: additional/panda_gazebo_gizem/description/panda_arm.urdf.xacro (robot description, xacro)
@@ -18,6 +18,6 @@
     <xacro:arg name="rpy" default="0 0 0" />
     <!-- Create a simulatable URDF -->
-    <xacro:include filename="$(find franka_description)/robots/utils.xacro" />
-    <xacro:include filename="$(find franka_description)/robots/panda_gazebo.xacro" />
+    <xacro:include filename="$(find panda_gazebo_gizem)/description/utils.xacro" />
+    <xacro:include filename="$(find panda_gazebo_gizem)/description/panda_gazebo.xacro" />
     <xacro:panda_arm arm_id="${arm_id}" />
     <xacro:if value="$(arg hand)">
@@ -40,14 +40,14 @@
     <xacro:gazebo-joint joint="${arm_id}_joint6" transmission="hardware_interface/EffortJointInterface" />
     <xacro:gazebo-joint joint="${arm_id}_joint7" transmission="hardware_interface/EffortJointInterface" />
-    <xacro:transmission-franka-state arm_id="${arm_id}" />
+    <!-- <xacro:transmission-franka-state arm_id="${arm_id}" />
     <xacro:transmission-franka-model arm_id="${arm_id}"
        root="${arm_id}_joint1"
        tip="${arm_id}_joint8"
-     />
+     /> -->
     <gazebo>
       <plugin name="gazebo_ros_control" filename="libgazebo_ros_control.so">
         <robotNamespace>${arm_id}</robotNamespace>
         <controlPeriod>0.001</controlPeriod>
-        <robotSimType>franka_gazebo/FrankaHWSim</robotSimType>
+        <robotSimType>gazebo_ros_control/DefaultRobotHWSim</robotSimType>
       </plugin>
       <self_collide>true</self_collide>

File: additional/panda_gazebo_gizem/description/utils.xacro (robot description, xacro)
@@ -7,5 +7,5 @@
   <!-- transmission - type of the transmission of the joint       -->
   <!-- ========================================================== -->
-  <xacro:macro name="gazebo-joint" params="joint transmission:=hardware_interface/EffortJointInterface">
+  <xacro:macro name="gazebo-joint" params="joint transmission:=hardware_interface/PositionJointInterface">
     <gazebo reference="${joint}">
       <!-- Needed for ODE to output external wrenches on joints -->
@@ -18,5 +18,6 @@
       </joint>
       <actuator name="${joint}_motor">
-        <hardwareInterface>${transmission}</hardwareInterface>
+        <!-- <hardwareInterface>${transmission}</hardwareInterface> -->
+        <mechanicalReduction>1</mechanicalReduction>
       </actuator>
     </transmission>
@@ -72,4 +73,23 @@
     </transmission>
   </xacro:macro>
+  <xacro:macro name="transmission-gizem-state" params="arm_id:=panda">
+    <transmission name="${arm_id}_gizem_state">
+      <type>franka_hw/FrankaStateInterface</type>
+      <joint name="${arm_id}_joint1"><hardwareInterface>franka_hw/FrankaStateInterface</hardwareInterface></joint>
+      <joint name="${arm_id}_joint2"><hardwareInterface>franka_hw/FrankaStateInterface</hardwareInterface></joint>
+      <joint name="${arm_id}_joint3"><hardwareInterface>franka_hw/FrankaStateInterface</hardwareInterface></joint>
+      <joint name="${arm_id}_joint4"><hardwareInterface>franka_hw/FrankaStateInterface</hardwareInterface></joint>
+      <joint name="${arm_id}_joint5"><hardwareInterface>franka_hw/FrankaStateInterface</hardwareInterface></joint>
+      <joint name="${arm_id}_joint6"><hardwareInterface>franka_hw/FrankaStateInterface</hardwareInterface></joint>
+      <joint name="${arm_id}_joint7"><hardwareInterface>franka_hw/FrankaStateInterface</hardwareInterface></joint>
+      <actuator name="${arm_id}_motor1"><hardwareInterface>franka_hw/FrankaStateInterface</hardwareInterface></actuator>
+      <actuator name="${arm_id}_motor2"><hardwareInterface>franka_hw/FrankaStateInterface</hardwareInterface></actuator>
+      <actuator name="${arm_id}_motor3"><hardwareInterface>franka_hw/FrankaStateInterface</hardwareInterface></actuator>
+      <actuator name="${arm_id}_motor4"><hardwareInterface>franka_hw/FrankaStateInterface</hardwareInterface></actuator>
+      <actuator name="${arm_id}_motor5"><hardwareInterface>franka_hw/FrankaStateInterface</hardwareInterface></actuator>
+      <actuator name="${arm_id}_motor6"><hardwareInterface>franka_hw/FrankaStateInterface</hardwareInterface></actuator>
+      <actuator name="${arm_id}_motor7"><hardwareInterface>franka_hw/FrankaStateInterface</hardwareInterface></actuator>
+    </transmission>
+  </xacro:macro>
   <!-- ============================================================ -->
   <!-- Adds the required tags to provide a `FrankaModelInterface`   -->
